File: Tabel Layout/SoftStart.kicad_sch (KiCad schematic)
At the start: 15 parts

Commit message: updates
Changed lines of the file:
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@@
 	(rectangle
 		(start 290.83 52.07)
-		(end 370.84 135.89)
+		(end 370.84 148.59)
 		(stroke
 			(width 1)
@@
 	)
 	(rectangle
-		(start 195.072 72.136)
-		(end 224.536 84.836)
+		(start 196.342 125.73)
+		(end 225.806 140.716)
 		(stroke
 			(width 0)
@@
 		)
 	)
+	(text "Thy Feedback\nGenerator"
+		(exclude_from_sim no)
+		(at 208.28 123.444 0)
+		(effects
+			(font
+				(size 1.27 1.27)
+			)
+		)
+	)
 	(text " 3 Phase Voltage \n    Generator"
 		(exclude_from_sim no)
@@
 		)
 	)
-	(text "Thy Feedback\nGenerator"
-		(exclude_from_sim no)
-		(at 203.454 78.74 0)
-		(effects
-			(font
-				(size 1.27 1.27)
-			)
-		)
+	(junction
+		(at 262.89 133.35)
+		(diameter 0)
+		(color 0 0 0 0)
 	)
 	(junction
@@
 	)
 	(junction
+		(at 269.24 128.27)
+		(diameter 0)
+		(color 0 0 0 0)
+	)
+	(junction
 		(at 275.59 68.58)
 		(diameter 0)
@@
 		(color 0 0 0 0)
 	)
+	(junction
+		(at 256.54 138.43)
+		(diameter 0)
+		(color 0 0 0 0)
+	)
 	(wire
 		(pts
@@
 	(wire
 		(pts
-			(xy 256.54 74.93) (xy 256.54 125.73)
+			(xy 256.54 74.93) (xy 256.54 138.43)
 		)
 		(stroke
@@
 	(wire
 		(pts
+			(xy 213.36 133.35) (xy 262.89 133.35)
+		)
+		(stroke
+			(width 0)
+			(type default)
+		)
+	)
+	(wire
+		(pts
+			(xy 213.36 138.43) (xy 256.54 138.43)
+		)
+		(stroke
+			(width 0)
+			(type default)
+		)
+	)
+	(wire
+		(pts
 			(xy 157.48 208.28) (xy 157.48 217.17)
 		)
 		(stroke
 			(width 0.4)
+			(type default)
+		)
+	)
+	(wire
+		(pts
+			(xy 269.24 128.27) (xy 294.64 128.27)
+		)
+		(stroke
+			(width 0)
 			(type default)
 		)
@@
 	(wire
 		(pts
-			(xy 262.89 80.01) (xy 262.89 125.73)
+			(xy 262.89 80.01) (xy 262.89 133.35)
 		)
 		(stroke
@@
 	(wire
 		(pts
+			(xy 213.36 128.27) (xy 269.24 128.27)
+		)
+		(stroke
+			(width 0)
+			(type default)
+		)
+	)
+	(wire
+		(pts
 			(xy 255.27 86.36) (xy 298.45 86.36)
 		)
@@
 	(wire
 		(pts
+			(xy 256.54 138.43) (xy 294.64 138.43)
+		)
+		(stroke
+			(width 0)
+			(type default)
+		)
+	)
+	(wire
+		(pts
 			(xy 151.13 204.47) (xy 151.13 213.36)
 		)
@@
 	(wire
 		(pts
-			(xy 269.24 83.82) (xy 269.24 125.73)
+			(xy 269.24 83.82) (xy 269.24 128.27)
 		)
 		(stroke
@@
 		(pts
 			(xy 275.59 64.77) (xy 275.59 68.58)
+		)
+		(stroke
+			(width 0)
+			(type default)
+		)
+	)
+	(wire
+		(pts
+			(xy 262.89 133.35) (xy 294.64 133.35)
 		)
 		(stroke
@@
 		)
 	)
+	(global_label "S_Motor"
+		(shape output)
+		(at 294.64 133.35 0)
+		(fields_autoplaced yes)
+		(effects
+			(font
+				(size 1.27 1.27)
+			)
+			(justify left)
+		)
+		(property "Intersheetrefs" "${INTERSHEET_REFS}"
+			(at 305.0636 133.35 0)
+			(effects
+				(font
+					(size 1.27 1.27)
+				)
+				(justify left)
+				(hide yes)
+			)
+		)
+	)
 	(global_label "Thy_S"
 		(shape output)
@@
 		)
 	)
+	(global_label "T_Motor"
+		(shape output)
+		(at 294.64 128.27 0)
+		(fields_autoplaced yes)
+		(effects
+			(font
+				(size 1.27 1.27)
+			)
+			(justify left)
+		)
+		(property "Intersheetrefs" "${INTERSHEET_REFS}"
+			(at 304.8217 128.27 0)
+			(effects
+				(font
+					(size 1.27 1.27)
+				)
+				(justify left)
+				(hide yes)
+			)
+		)
+	)
 	(global_label "C_S"
 		(shape input)
@@
 		)
 	)
-	(global_label "Thy_R_FB"
-		(shape output)
-		(at 212.09 74.93 0)
-		(fields_autoplaced yes)
-		(effects
-			(font
-				(size 1.27 1.27)
-			)
-			(justify left)
-		)
-		(property "Intersheetrefs" "${INTERSHEET_REFS}"
-			(at 223.7232 74.93 0)
-			(effects
-				(font
-					(size 1.27 1.27)
-				)
-				(justify left)
-				(hide yes)
-			)
-		)
-	)
 	(global_label "V_R"
 		(shape output)
@@
 		)
 	)
+	(global_label "R_Motor"
+		(shape output)
+		(at 294.64 138.43 0)
+		(fields_autoplaced yes)
+		(effects
+			(font
+				(size 1.27 1.27)
+			)
+			(justify left)
+		)
+		(property "Intersheetrefs" "${INTERSHEET_REFS}"
+			(at 305.1241 138.43 0)
+			(effects
+				(font
+					(size 1.27 1.27)
+				)
+				(justify left)
+				(hide yes)
+			)
+		)
+	)
 	(global_label "C_T"
 		(shape output)
@@
 		)
 	)
-	(global_label "T"
-		(shape output)
-		(at 269.24 125.73 270)
-		(fields_autoplaced yes)
-		(effects
-			(font
-				(size 1.27 1.27)
-			)
-			(justify right)
-		)
-		(property "Intersheetrefs" "${INTERSHEET_REFS}"
-			(at 269.24 129.6828 90)
-			(effects
-				(font
-					(size 1.27 1.27)
-				)
-				(justify right)
-				(hide yes)
-			)
-		)
-	)
 	(global_label "V_S"
 		(shape output)
@@
 		)
 	)
-	(global_label "R"
-		(shape output)
-		(at 256.54 125.73 270)
-		(fields_autoplaced yes)
-		(effects
-			(font
-				(size 1.27 1.27)
-			)
-			(justify right)
-		)
-		(property "Intersheetrefs" "${INTERSHEET_REFS}"
-			(at 256.54 129.9852 90)
-			(effects
-				(font
-					(size 1.27 1.27)
-				)
-				(justify right)
-				(hide yes)
-			)
-		)
-	)
 	(global_label "V_R"
 		(shape input)
@@
 		)
 	)
-	(global_label "S"
-		(shape output)
-		(at 262.89 125.73 270)
-		(fields_autoplaced yes)
-		(effects
-			(font
-				(size 1.27 1.27)
-			)
-			(justify right)
-		)
-		(property "Intersheetrefs" "${INTERSHEET_REFS}"
-			(at 262.89 129.9247 90)
-			(effects
-				(font
-					(size 1.27 1.27)
-				)
-				(justify right)
-				(hide yes)
-			)
-		)
-	)
 	(global_label "Thy_R"
 		(shape input)
@@
 		)
 	)
+	(global_label "Thy_R_FB"
+		(shape input)
+		(at 213.36 138.43 180)
+		(fields_autoplaced yes)
+		(effects
+			(font
+				(size 1.27 1.27)
+			)
+			(justify right)
+		)
+		(property "Intersheetrefs" "${INTERSHEET_REFS}"
+			(at 201.7268 138.43 0)
+			(effects
+				(font
+					(size 1.27 1.27)
+				)
+				(justify right)
+				(hide yes)
+			)
+		)
+	)
 	(global_label "C_S"
 		(shape output)
@@
 		)
 	)
+	(global_label "Thy_S_FB"
+		(shape input)
+		(at 213.36 133.35 180)
+		(fields_autoplaced yes)
+		(effects
+			(font
+				(size 1.27 1.27)
+			)
+			(justify right)
+		)
+		(property "Intersheetrefs" "${INTERSHEET_REFS}"
+			(at 201.7873 133.35 0)
+			(effects
+				(font
+					(size 1.27 1.27)
+				)
+				(justify right)
+				(hide yes)
+			)
+		)
+	)
 	(global_label "Thy_T_FB"
-		(shape output)
-		(at 212.09 82.55 0)
-		(fields_autoplaced yes)
-		(effects
-			(font
-				(size 1.27 1.27)
-			)
-			(justify left)
-		)
-		(property "Intersheetrefs" "${INTERSHEET_REFS}"
-			(at 223.4208 82.55 0)
-			(effects
-				(font
-					(size 1.27 1.27)
-				)
-				(justify left)
-				(hide yes)
-			)
-		)
-	)
-	(global_label "Thy_S_FB"
-		(shape output)
-		(at 212.09 78.74 0)
-		(fields_autoplaced yes)
-		(effects
-			(font
-				(size 1.27 1.27)
-			)
-			(justify left)
-		)
-		(property "Intersheetrefs" "${INTERSHEET_REFS}"
-			(at 223.6627 78.74 0)
-			(effects
-				(font
-					(size 1.27 1.27)
-				)
-				(justify left)
-				(hide yes)
-			)
+		(shape input)
+		(at 213.36 128.27 180)
+		(fields_autoplaced yes)
+		(effects
+			(font
+				(size 1.27 1.27)
+			)
+			(justify right)
+		)
+		(property "Intersheetrefs" "${INTERSHEET_REFS}"
+			(at 202.0292 128.27 0)
+			(effects
+				(font
+					(size 1.27 1.27)
+				)
+				(justify right)
+				(hide yes)
+			)
