File: Tabel Layout/SS_Topology.kicad_sch (KiCad schematic)
At the start: 30 parts, among them Q1 TIC106, Q2 TIC106, Q3 TIC106, Q4 TIC106, Q5 TIC106, Q6 TIC106

Commit message: updates
Parts:
- added C1, C2, C3: C, symbol Device:C
- added R10, R11, R12: R, symbol Device:R
Connections:
- net R: now also C1.1
- net S: now also C2.1
- net T: now also C3.1
- net at D6.2 (A), Q3.1 (K), Q4.2 (A): now also R11.2
- net at D5.2 (A), Q5.1 (K), Q6.2 (A): now also R12.2
- net at D1.2 (A), Q1.2 (A), Q2.1 (K): now also R10.2
- new net: C1.2, R10.1
- new net: C2.2, R11.1
- new net: C3.2, R12.1
Other:
- note added: "Snubber"
- title: (none) -> Soft Starter Topology

Commit message: updates
Changed lines of the file:
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@@
 	)
 	(junction
-		(at 190.5 73.66)
+		(at 288.29 48.26)
 		(diameter 0)
 		(color 0 0 0 0)
 	)
 	(junction
-		(at 214.63 107.95)
+		(at 190.5 73.66)
 		(diameter 0)
 		(color 0 0 0 0)
 	)
 	(junction
-		(at 280.67 44.45)
+		(at 214.63 107.95)
 		(diameter 0)
 		(color 0 0 0 0)
 	)
 	(junction
-		(at 237.49 149.86)
+		(at 280.67 44.45)
 		(diameter 0)
 		(color 0 0 0 0)
 	)
 	(junction
-		(at 288.29 48.26)
+		(at 237.49 149.86)
 		(diameter 0)
 		(color 0 0 0 0)
@@
 	)
 	(junction
-		(at 295.91 52.07)
+		(at 294.64 52.07)
 		(diameter 0)
 		(color 0 0 0 0)
@@
 		)
 	)
+	(wire
+		(pts
+			(xy 288.29 48.26) (xy 344.17 48.26)
+		)
+		(stroke
+			(width 0)
+			(type default)
+		)
+	)
 	(polyline
 		(pts
@@
 	(wire
 		(pts
+			(xy 288.29 48.26) (xy 288.29 72.39)
+		)
+		(stroke
+			(width 0)
+			(type default)
+		)
+	)
+	(wire
+		(pts
 			(xy 222.25 219.71) (xy 228.6 214.63)
 		)
@@
 	(wire
 		(pts
-			(xy 190.5 163.83) (xy 280.67 163.83)
-		)
-		(stroke
-			(width 0)
-			(type default)
-		)
-	)
-	(wire
-		(pts
 			(xy 215.9 101.6) (xy 214.63 101.6)
 		)
@@
 	(wire
 		(pts
+			(xy 237.49 156.21) (xy 273.05 156.21)
+		)
+		(stroke
+			(width 0)
+			(type default)
+		)
+	)
+	(wire
+		(pts
 			(xy 190.5 87.63) (xy 190.5 88.9)
 		)
@@
 	(wire
 		(pts
-			(xy 215.9 160.02) (xy 280.67 160.02)
-		)
-		(stroke
-			(width 0)
-			(type default)
-		)
-	)
-	(wire
-		(pts
 			(xy 231.14 114.3) (xy 273.05 114.3)
 		)
@@
 		)
 	)
-	(wire
+	(polyline
 		(pts
-			(xy 295.91 52.07) (xy 295.91 90.17)
+			(xy 59.436 38.862) (xy 89.662 38.862)
 		)
 		(stroke
@@
 	(polyline
 		(pts
-			(xy 59.436 38.862) (xy 89.662 38.862)
+			(xy 57.658 53.594) (xy 59.436 51.054)
 		)
 		(stroke
@@
 		)
 	)
-	(polyline
+	(wire
 		(pts
-			(xy 57.658 53.594) (xy 59.436 51.054)
+			(xy 215.9 160.02) (xy 215.9 219.71)
 		)
 		(stroke
-			(width 0)
+			(width 1)
 			(type default)
 		)
@@
 	(wire
 		(pts
-			(xy 215.9 160.02) (xy 215.9 219.71)
+			(xy 215.9 160.02) (xy 273.05 160.02)
 		)
 		(stroke
-			(width 1)
+			(width 0)
 			(type default)
 		)
@@
 	(wire
 		(pts
-			(xy 295.91 52.07) (xy 344.17 52.07)
+			(xy 237.49 52.07) (xy 294.64 52.07)
 		)
 		(stroke
@@
 		)
 	)
-	(wire
-		(pts
-			(xy 237.49 156.21) (xy 280.67 156.21)
-		)
-		(stroke
-			(width 0)
-			(type default)
-		)
-	)
 	(polyline
 		(pts
@@
 	(wire
 		(pts
+			(xy 294.64 52.07) (xy 294.64 72.39)
+		)
+		(stroke
+			(width 0)
+			(type default)
+		)
+	)
+	(wire
+		(pts
 			(xy 214.63 107.95) (xy 217.17 107.95)
 		)
@@
 		)
 	)
+	(wire
+		(pts
+			(xy 294.64 52.07) (xy 344.17 52.07)
+		)
+		(stroke
+			(width 0)
+			(type default)
+		)
+	)
+	(wire
+		(pts
+			(xy 190.5 163.83) (xy 273.05 163.83)
+		)
+		(stroke
+			(width 0)
+			(type default)
+		)
+	)
 	(polyline
 		(pts
@@
 	(wire
 		(pts
-			(xy 280.67 44.45) (xy 280.67 90.17)
+			(xy 280.67 44.45) (xy 280.67 72.39)
 		)
 		(stroke
@@
 	(wire
 		(pts
-			(xy 288.29 48.26) (xy 288.29 90.17)
-		)
-		(stroke
-			(width 0)
-			(type default)
-		)
-	)
-	(wire
-		(pts
 			(xy 179.07 92.71) (xy 190.5 92.71)
 		)
@@
 	(wire
 		(pts
-			(xy 295.91 52.07) (xy 237.49 52.07)
-		)
-		(stroke
-			(width 0)
-			(type default)
-		)
-	)
-	(wire
-		(pts
 			(xy 204.47 121.92) (xy 215.9 121.92)
 		)
@@
 	(wire
 		(pts
-			(xy 288.29 48.26) (xy 344.17 48.26)
-		)
-		(stroke
-			(width 0)
-			(type default)
-		)
-	)
-	(wire
-		(pts
 			(xy 187.96 168.91) (xy 273.05 168.91)
 		)
@@
 		)
 		(property "Value" "R"
-			(at 176.276 86.106 0)
+			(at 180.34 86.36 0)
 			(effects
 				(font
@@
 		)
 		(property "Value" "R"
-			(at 201.168 115.57 0)
+			(at 206.248 116.078 0)
 			(effects
 				(font
@@
 		)
 		(property "Value" "C"
-			(at 202.438 111.506 0)
+			(at 205.994 112.014 0)
 			(effects
 				(font
@@
 		)
 		(property "Value" "R"
-			(at 224.536 143.256 0)
+			(at 228.854 143.51 0)
 			(effects
 				(font
@@
 		)
 		(property "Value" "C"
-			(at 225.298 138.176 0)
+			(at 228.092 138.43 0)
 			(effects
 				(font
@@
 		)
 		(property "Value" "C"
-			(at 177.038 81.026 0)
+			(at 179.832 81.28 0)
 			(effects
 				(font
