File: Cur_Emul/Cur_Emul.kicad_pcb (KiCad board)
At the start: 2 copper layers, 570.6 x 233.2 mm, 476 parts, among them J1 Screw_Terminal_01x01, J10 Screw_Terminal_01x01, J11 Screw_Terminal_01x01, J12 Screw_Terminal_01x01, J13 Screw_Terminal_01x01, J14 Screw_Terminal_01x01, J15 Screw_Terminal_01x01, J16 Screw_Terminal_01x01, J17 Conn_01x04_Pin, J18 Conn_01x02_Pin, J19 Conn_01x04_Pin, J2 Screw_Terminal_01x01, J20 Conn_01x04_Pin, J21 Screw_Terminal_01x01, J22 Screw_Terminal_01x01, J23 Conn_01x06_Pin, J24 Conn_01x08_Pin, J25 Conn_01x08_Pin, J26 Conn_01x04_Pin, J27 Conn_01x04_Pin, J28 Conn_01x03_Pin, J28 Conn_01x04_Pin, J29 Conn_01x02_Pin, J3 Screw_Terminal_01x01, J30 Conn_01x02_Pin, J31 Conn_01x02_Pin, J32 Conn_01x04_Pin, J33 Conn_01x08_Pin, J34 Conn_01x06_Pin, J35 Conn_01x04_Pin, J36 Conn_01x06_Pin, J37 Conn_01x02_Pin, J38 Conn_01x02_Pin, J39 Conn_01x02_Pin, J4 Screw_Terminal_01x01, J40 Conn_01x01_Pin, J41 Conn_01x01_Pin, J42 Conn_01x01_Pin, J43 Conn_01x01_Pin, J44 Conn_01x01_Pin, J45 Conn_01x01_Pin, J46 Conn_01x01_Pin, J47 Conn_01x01_Pin, J48 Conn_01x01_Pin, J5 Screw_Terminal_01x01, J6 Screw_Terminal_01x01, J7 Screw_Terminal_01x01, J8 Screw_Terminal_01x01, J9 Screw_Terminal_01x01, M1 IXTH64N10L2, M10 IRF530, M11 IRF530, M12 IRF530, M2 IXTH64N10L2, M3 IXTH64N10L2, M4 IXTH64N10L2, M5 IXTH64N10L2, M6 IXTH64N10L2, M7 IRF530, M8 IRF530, M9 IRF530, T1 Transformer_1P_2S, T2 Transformer_1P_2S, T3 Transformer_1P_2S, U1 Opamp_Quad, U10 Opamp_Quad, U11 Opamp_Quad, U12 Opamp_Quad, U13 LM317_SOT-223, U14 LM317_SOT-223, U14 TLP3023, U15 LM7812_TO220, U16 TLP3023, U17 SFH6206-2T, U18 TLP3023, U19 SFH6206-2T, U2 Opamp_Quad, U20 SFH6206-2T, U3 Opamp_Quad, U4 Opamp_Quad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

Commit message: updates
Parts:
- removed the J28 at (-43.2, 98.9)
- removed the JP11 at (-102.3, 134.3)
- removed the U14 at (-35.8, 123.2)
- added D18: LED, LED_SMD:LED_0805_2012Metric_Pad1.15x1.40mm_HandSolder, F.Cu at (450.0, 204.0)
- added D23: LED, LED_SMD:LED_0805_2012Metric_Pad1.15x1.40mm_HandSolder, F.Cu at (450.0, 195.0)
- added J31: Conn_01x02_Pin, Connector_Phoenix_GMSTB:PhoenixContact_GMSTBA_2,5_2-G_1x02_P7.50mm_Horizontal, F.Cu at (27.8, 68.8)
- added J36: Conn_01x08_Pin, Connector_JST:JST_PH_B8B-PH-K_1x08_P2.00mm_Vertical, F.Cu at (723.5, 16.9)
- added J49: Conn_01x04_Pin, Connector_Phoenix_GMSTB:PhoenixContact_GMSTBA_2,5_4-G-7,62_1x04_P7.62mm_Horizontal, F.Cu at (36.1, 171.2)
- added J50: Conn_01x04_Pin, Connector_Phoenix_GMSTB:PhoenixContact_GMSTBA_2,5_4-G-7,62_1x04_P7.62mm_Horizontal, F.Cu at (439.2, 186.3)
- added J51: Conn_01x02_Pin, Connector_Phoenix_GMSTB:PhoenixContact_GMSTBA_2,5_2-G_1x02_P7.50mm_Horizontal, F.Cu at (437.3, 91.8)
- added J52: Conn_01x02_Pin, Connector_Phoenix_GMSTB:PhoenixContact_GMSTBA_2,5_2-G_1x02_P7.50mm_Horizontal, F.Cu at (437.3, 111.8)
- added J53: Conn_01x02_Pin, Connector_Phoenix_GMSTB:PhoenixContact_GMSTBA_2,5_2-G_1x02_P7.50mm_Horizontal, F.Cu at (392.7, 102.8)
- added J54: Conn_01x02_Pin, Connector_Phoenix_GMSTB:PhoenixContact_GMSTBA_2,5_2-G_1x02_P7.50mm_Horizontal, F.Cu at (392.7, 121.8)
- added R171: 220R, Resistor_THT:R_Axial_DIN0207_L6.3mm_D2.5mm_P7.62mm_Horizontal, F.Cu at (722.1, -16.2)
- added R172: 220R, Resistor_THT:R_Axial_DIN0207_L6.3mm_D2.5mm_P7.62mm_Horizontal, F.Cu at (491.2, 7.50)
- added R194: 220R, Resistor_THT:R_Axial_DIN0207_L6.3mm_D2.5mm_P7.62mm_Horizontal, F.Cu at (722.1, -8.12)
- added R195: 220R, Resistor_THT:R_Axial_DIN0207_L6.3mm_D2.5mm_P7.62mm_Horizontal, F.Cu at (491.2, 15.6)
- added R200: 10K, Resistor_THT:R_Axial_DIN0207_L6.3mm_D2.5mm_P7.62mm_Horizontal, F.Cu at (722.1, -0.02)
- added R202: 33K, Resistor_THT:R_Axial_DIN0207_L6.3mm_D2.5mm_P7.62mm_Horizontal, F.Cu at (722.1, 4.03)
- added R204: 33K, Resistor_THT:R_Axial_DIN0207_L6.3mm_D2.5mm_P7.62mm_Horizontal, F.Cu at (722.1, 8.08)
- added R208: 10K, Resistor_THT:R_Axial_DIN0207_L6.3mm_D2.5mm_P7.62mm_Horizontal, F.Cu at (722.1, 12.1)
- added R210: 10K, Resistor_THT:R_Axial_DIN0207_L6.3mm_D2.5mm_P7.62mm_Horizontal, F.Cu at (732.8, -16.2)
- added R212: 220R, Resistor_THT:R_Axial_DIN0207_L6.3mm_D2.5mm_P7.62mm_Horizontal, F.Cu at (502.0, 7.50)
- added R215: 5K, Resistor_SMD:R_0805_2012Metric_Pad1.20x1.40mm_HandSolder, F.Cu at (455.0, 204.0)
- added R216: 5K, Resistor_SMD:R_0805_2012Metric_Pad1.20x1.40mm_HandSolder, F.Cu at (452.5, 204.0)
- added R217: 5K, Resistor_SMD:R_0805_2012Metric_Pad1.20x1.40mm_HandSolder, F.Cu at (455.0, 195.0)
- added R218: 5K, Resistor_SMD:R_0805_2012Metric_Pad1.20x1.40mm_HandSolder, F.Cu at (452.5, 195.0)
- added R219: 10K, Resistor_THT:R_Axial_DIN0207_L6.3mm_D2.5mm_P7.62mm_Horizontal, F.Cu at (732.8, -8.12)
- added R220: 33K, Resistor_THT:R_Axial_DIN0207_L6.3mm_D2.5mm_P7.62mm_Horizontal, F.Cu at (732.8, -4.07)
- added R221: 33K, Resistor_THT:R_Axial_DIN0207_L6.3mm_D2.5mm_P7.62mm_Horizontal, F.Cu at (732.8, -0.02)
- added R222: 33K, Resistor_THT:R_Axial_DIN0207_L6.3mm_D2.5mm_P7.62mm_Horizontal, F.Cu at (732.8, 4.03)
- added R223: 33K, Resistor_THT:R_Axial_DIN0207_L6.3mm_D2.5mm_P7.62mm_Horizontal, F.Cu at (732.8, 8.08)
- added R224: 220R, Resistor_THT:R_Axial_DIN0207_L6.3mm_D2.5mm_P7.62mm_Horizontal, F.Cu at (732.8, 12.1)
- added R225: 33K, Resistor_THT:R_Axial_DIN0207_L6.3mm_D2.5mm_P7.62mm_Horizontal, F.Cu at (743.6, -16.2)
- added R226: 33K, Resistor_THT:R_Axial_DIN0207_L6.3mm_D2.5mm_P7.62mm_Horizontal, F.Cu at (743.6, -12.2)
- added R227: 10K, Resistor_THT:R_Axial_DIN0207_L6.3mm_D2.5mm_P7.62mm_Horizontal, F.Cu at (743.6, -8.12)
- added R228: 33K, Resistor_THT:R_Axial_DIN0207_L6.3mm_D2.5mm_P7.62mm_Horizontal, F.Cu at (743.6, -4.07)
- added R229: 33K, Resistor_THT:R_Axial_DIN0207_L6.3mm_D2.5mm_P7.62mm_Horizontal, F.Cu at (743.6, -0.02)
- added R230: 33K, Resistor_THT:R_Axial_DIN0207_L6.3mm_D2.5mm_P7.62mm_Horizontal, F.Cu at (743.6, 4.03)
- added R231: 33K, Resistor_THT:R_Axial_DIN0207_L6.3mm_D2.5mm_P7.62mm_Horizontal, F.Cu at (743.6, 8.08)
- added TP73: TestPoint_Alt, TestPoint:TestPoint_Loop_D1.80mm_Drill1.0mm_Beaded, F.Cu at (46.2, 139.5)
- added TP74: TestPoint_Alt, TestPoint:TestPoint_Loop_D1.80mm_Drill1.0mm_Beaded, F.Cu at (705.8, 17.4)
- added TP75: TestPoint_Alt, TestPoint:TestPoint_Loop_D1.80mm_Drill1.0mm_Beaded, F.Cu at (705.8, 22.0)
- added TP76: TestPoint_Alt, TestPoint:TestPoint_Loop_D1.80mm_Drill1.0mm_Beaded, F.Cu at (705.8, 26.7)
- added U21: SFH6206-2T, Package_DIP:SMDIP-4_W9.53mm_Clearance8mm, F.Cu at (746.7, 17.5)
- added U22: SFH6206-2T, Package_DIP:SMDIP-4_W9.53mm_Clearance8mm, F.Cu at (746.7, 24.1)
- added U23: SFH6206-2T, Package_DIP:SMDIP-4_W9.53mm_Clearance8mm, F.Cu at (746.7, 30.7)
- C48: footprint Capacitor_SMD:CP_Elec_6.3x7.7 -> Capacitor_THT:CP_Radial_D24.0mm_P10.00mm_SnapIn
- D1: value NRVA4004T3G -> 1N4007; footprint Diode_SMD:D_SMA -> Diode_THT:D_DO-41_SOD81_P10.16mm_Horizontal
- J19, J27, J32: value Conn_01x04_Pin -> Conn_01x02_Pin; footprint Connector_JST:JST_EH_B4B-EH-A_1x04_P2.50mm_Vertical -> Connector_Phoenix_GMSTB:PhoenixContact_GMSTBVA_2,5_2-G_1x02_P7.50mm_Vertical
- R158, R44, R48: footprint Resistor_SMD:R_1206_3216Metric_Pad1.30x1.75mm_HandSolder -> Resistor_THT:R_Axial_DIN0204_L3.6mm_D1.6mm_P7.62mm_Horizontal
- R159, R160, R47: footprint Resistor_SMD:R_1206_3216Metric_Pad1.30x1.75mm_HandSolder -> Resistor_SMD:R_Shunt_Vishay_WSR2_WSR3
- R161, R164: value 1K -> 5K
- moved C52 614.4 mm to (978.0, -228.0), turned to -90 degrees
- moved TP60 604.3 mm to (503.0, 146.5), turned to -90 degrees
- moved C51 584.2 mm to (909.5, -250.0), turned to -90 degrees
- moved J34 557.6 mm to (886.5, -160.5)
- moved R207 547.5 mm to (990.7, -231.9), turned to -90 degrees
- moved R208 546.8 mm to (986.6, -231.9), turned to -90 degrees
- moved R209 539.1 mm to (1019.0, -221.1), turned to -90 degrees
- moved R210 537.9 mm to (1015.0, -221.1), turned to -90 degrees
- moved R211 536.9 mm to (1011.0, -221.1), turned to -90 degrees
- moved R213 534.9 mm to (1002.9, -221.1), turned to -90 degrees
- moved R214 534.0 mm to (998.8, -221.1), turned to -90 degrees
- moved TP72 520.5 mm to (1009.5, -209.6), turned to -90 degrees
- moved U15 499.5 mm to (436.4, 147.5)
- moved C50 493.0 mm to (764.0, -235.3), turned to -90 degrees
- moved JP21 492.4 mm to (436.5, 130.5)
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Connections:
- C3 pad 1: +3.3V -> +15V
- C31 pad 2: GND -> GND2
- C32 pad 2: GND -> GND2
- C35 pad 2: GND -> GND2
- C36 pad 2: GND -> GND2
- C37 pad 1: +15V -> +12VA
- C37 pad 2: GND -> GND2
- C38 pad 1: +15V -> +12VA
- C38 pad 2: GND -> GND2
- C39 pad 1: +15V -> +12VA
- C39 pad 2: GND -> GND2
- C40 pad 1: +15V -> +12VA
- C40 pad 2: GND -> GND2
- C41 pad 1: +15V -> +12VA
- C41 pad 2: GND -> GND2
- C42 pad 1: +15V -> +12VA
- C42 pad 2: GND -> GND2
- C43 pad 1: +15V -> +12VA
- C43 pad 2: GND -> GND2
- C44 pad 1: +15V -> +12VA
- C44 pad 2: GND -> GND2
- C45 pad 1: +15V -> +12VA
- C45 pad 2: GND -> GND2
- C46 pad 1: +15V -> +12VA
- C46 pad 2: GND -> GND2
- C47 pad 1: +15V -> +3.3V
- C48 pad 2: GND -> GND2
- C5 pad 2: GND -> GND2
- C50 pad 2: GND -> GND2
- C51 pad 2: GND -> GND2
- C52 pad 2: GND -> GND2
- C6 pad 2: GND -> GND2
- D17 pad 1: GND -> GNDPWR
- D2 pad 1: GND -> GND2
- J19 pad 1: R_Prim_H -> Net-(J19-Pin_1)
- J19 pad 2: R_Volt_Lim -> Net-(J19-Pin_2)
- J27 pad 1: T_Prim_H -> Net-(J27-Pin_1)
- J27 pad 2: T_Volt_Lim -> Net-(J27-Pin_2)
- J32 pad 1: S_Prim_H -> Net-(J32-Pin_1)
- J32 pad 2: S_Volt_Lim -> Net-(J32-Pin_2)
- J33 pad 3: S_Volt_PWM_L -> S_Volt_PWM_H
- J33 pad 4: S_Volt_PWM_H -> S_Volt_PWM_L
- J33 pad 7: GND -> GND2
- J33 pad 8: GND -> GND2
- J34 pad 1: GND -> GND2
- J34 pad 2: GND -> GND2
- J35 pad 1: GND -> GND2
- J36 pad 1: GND -> GND2
- J36 pad 2: GND -> GND2
- J36 pad 6: +3.3V -> +3.3VA
- JP10 pad 3: GND -> GND2
- JP14 pad 3: GND -> GND2
- JP16 pad 3: GND -> GND2
- JP17 pad 3: GND -> GND2
- JP18 pad 3: GND -> GND2
- JP19 pad 3: GND -> GND2
- JP21 pad 1: Net-(J31-Pin_1) -> Net-(J51-Pin_1)
- JP21 pad 3: VBUS -> Net-(J52-Pin_1)
- R103 pad 2: +3.3V -> +3.3VA
- R107 pad 2: +3.3V -> +3.3VA
- R111 pad 2: +3.3V -> +3.3VA
- R112 pad 2: GND -> GND2
- R114 pad 2: +3.3V -> +3.3VA
- R115 pad 2: GND -> GND2
- R120 pad 1: GND -> GND2
- R121 pad 1: GND -> GND2
- R131 pad 2: +3.3V -> +3.3VA
- R132 pad 2: GND -> GND2
- R134 pad 2: +3.3V -> +3.3VA
- R135 pad 2: GND -> GND2
- R140 pad 1: GND -> GND2
- R141 pad 1: GND -> GND2
- R150 pad 1: +15V -> +12VA
- R151 pad 1: GND -> GND2
- R152 pad 1: +15V -> +12VA
- R153 pad 1: GND -> GND2
- R155 pad 2: +15V -> +3.3V
- R156 pad 1: Net-(R156-Pad1) -> Net-(U7-ADJ)
- R156 pad 2: +3.3V -> +15V
- R157 pad 2: Net-(R156-Pad1) -> Net-(U7-ADJ)
- R158 pad 2: GND -> GND2
- R159 pad 2: GND -> GND2
- R160 pad 2: GND -> GND2
- R162 pad 2: +3.3V -> +15V
- R163 pad 2: +15V -> +3.3V
- R167 pad 1: Net-(R167-Pad1) -> V1_Line
- R168 pad 2: Notr -> V1_Motor
- R169 pad 1: Net-(R169-Pad1) -> V2_Line
- R170 pad 2: Notr -> V2_Motor
- R177 pad 2: Net-(R177-Pad2) -> Net-(J37-Pin_1)
- R178 pad 1: Net-(R177-Pad2) -> Net-(R178-Pad1)
- R180 pad 1: R_Phase_Ret -> R1_Fire
- R180 pad 2: +3.3V -> +3.3VA
- R181 pad 1: T_Phase_Ret -> T1_Fire
- R181 pad 2: +3.3V -> +3.3VA
- R183 pad 2: Net-(R183-Pad2) -> Net-(J38-Pin_1)
- R184 pad 1: Net-(R183-Pad2) -> Net-(R184-Pad1)
- R186 pad 1: S_Phase_Ret -> S1_Fire
- R186 pad 2: +3.3V -> +3.3VA
- R188 pad 2: Net-(R188-Pad2) -> Net-(J39-Pin_1)
- R189 pad 1: Net-(R188-Pad2) -> Net-(R189-Pad1)
- R191 pad 2: GND -> GND2
- R193 pad 1: GND -> GND2
- R204 pad 1: GND -> GND2
- R205 pad 2: GND -> GND2
- R212 pad 1: GND -> GND2
- R213 pad 2: GND -> GND2
- R44 pad 2: GND -> GND2
- R47 pad 2: GND -> GND2
- R48 pad 2: GND -> GND2
- R49 pad 1: GND -> GND2
- R94 pad 2: GND -> GND2
- R95 pad 2: GND -> GND2
- R96 pad 1: GND -> GND2
- T1 pad 1: R_Sec_b -> R_Sec_a
- T1 pad 10: R_Prim_H -> R_Prim_L
- T1 pad 5: R_Sec_a -> R_Sec_b
- T1 pad 6: R_Prim_L -> R_Prim_H
- T2 pad 1: T_Sec_b -> T_Sec_a
- T2 pad 10: T_Prim_H -> T_Prim_L
- T2 pad 5: T_Sec_a -> T_Sec_b
- T2 pad 6: T_Prim_L -> T_Prim_H
- T3 pad 1: S_Sec_b -> S_Sec_a
- T3 pad 10: S_Prim_H -> S_Prim_L
- T3 pad 5: S_Sec_a -> S_Sec_b
- T3 pad 6: S_Prim_L -> S_Prim_H
- TP17 pad 1: GND -> GND2
- TP38 pad 1: +3.3V -> +15V
- TP59 pad 1: +15V -> +3.3V
- TP64 pad 1: T_Phase_Ret -> T1_Fire
- TP65 pad 1: R_Phase_Ret -> R1_Fire
- TP66 pad 1: S_Phase_Ret -> S1_Fire
- TP67 pad 1: GND -> GND2
- TP68 pad 1: GND -> GND2
- TP69 pad 1: GND -> GND2
- U10 pad 11: GND -> GND2
- U10 pad 4: +15V -> +12VA
- U11 pad 11: GND -> GND2
- U11 pad 4: +15V -> +12VA
- U12 pad 11: GND -> GND2
- U12 pad 4: +15V -> +12VA
- U13 pad 2: +15V -> +3.3V
- U14 pad 2: GND -> GND2
- U14 pad 4: Net-(R167-Pad1) -> Net-(R195-Pad1)
- U14 pad 6: R_Sec_b -> V1_Motor
- U15 pad 2: GND -> GND2
- U16 pad 2: GND -> GND2
- U16 pad 4: Net-(R169-Pad1) -> Net-(R172-Pad1)
- U16 pad 6: S_Sec_b -> V2_Motor
- U17 pad 2: Net-(J37-Pin_1) -> Net-(R178-Pad1)
- U17 pad 3: GND -> GND2
- U17 pad 4: R_Phase_Ret -> R1_Fire
- U18 pad 2: GND -> GND2
- U18 pad 4: Net-(R171-Pad1) -> Net-(R212-Pad1)
- U18 pad 6: T_Sec_b -> V3_Motor
- U19 pad 2: Net-(J38-Pin_1) -> Net-(R184-Pad1)
- U19 pad 3: GND -> GND2
- U19 pad 4: T_Phase_Ret -> T1_Fire
- U20 pad 2: Net-(J39-Pin_1) -> Net-(R189-Pad1)
- U20 pad 3: GND -> GND2
- U20 pad 4: S_Phase_Ret -> S1_Fire
- U7 pad 1: GND -> Net-(U7-ADJ)
- U7 pad 2: +3.3V -> +15V
- U8 pad 11: GND -> GND2
- U8 pad 4: +15V -> +12VA
- U9 pad 11: GND -> GND2
- U9 pad 4: +15V -> +12VA
Routing:
- net GND2: track 0.00 -> 1226.2 mm, vias 0 -> 14
- net VBUS: track 0.00 -> 1157.7 mm, vias 0 -> 5
- net GND: track 105.1 -> 949.2 mm, vias 0 -> 22
- net +15V: track 20.9 -> 414.3 mm, vias 0 -> 6
- net +12VA: track 0.00 -> 344.1 mm, vias 0 -> 2
- net Net-(J3-Pin_1): track 0.00 -> 323.4 mm
- net +3.3V: track 118.1 -> 438.9 mm
- net VDD: track 0.00 -> 316.2 mm
- net GNDPWR: track 0.00 -> 211.3 mm
- net Net-(JP9-A): track 0.00 -> 206.2 mm
- net R_PWM_Analog: track 5.69 -> 175.9 mm, vias 0 -> 2
- net R_Tot_I: track 4.51 -> 166.8 mm, vias 0 -> 1
- net S_Mos_I_1: track 0.00 -> 158.5 mm, vias 0 -> 1
- net T_Tot_I: track 0.00 -> 145.1 mm
- net T_Sec_a: track 0.00 -> 136.6 mm
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- added copper zone on B.Cu, net GND
- added copper zone on F.Cu, net GND
Other:
- board size 570.6 x 233.2 mm -> 656.3 x 217.1 mm
- board text added: "15V"
- board text added: "3V3"
- board text added: "3V3 Input Bus/Ext"
- board text added: "CS1"
- board text added: "CS2"
- board text added: "CURRENT GENERATOR"
- board text added: "DC BUS"
- board text added: "LDAC1"
- board text added: "LDAC2"
- board text added: "R-ANALOG_INP"
- board text added: "R-AnalogGain"
- board text added: "R-MOS1 Currrent None/Limit JP1"
- board text added: "R-MOS2 Current None/Limit"
- board text added: "R-Mos1_Drive"
- board text added: "R-Mos2_Drive"
- board text added: "R-PWM/ANALOG"
- board text added: "R-Tot_Current"
- board text added: "S-ANALOG_INP"
- board text added: "S-AnalogGain"
- board text added: "S-MOS1 Current None/Limit"
- board text added: "S-MOS2 Current None/Limit"
- board text added: "S-Mos1_Drive"
- board text added: "S-Mos2_Drive"
- board text added: "S-PWM/ANALOG"
- board text added: "S-Tot_Current"
- board text added: "SCK1"
- board text added: "SCK2"
- board text added: "SDI1"
- board text added: "SDI2"
- board text added: "T-ANALOG_INP"
- board text added: "T-AnalogGain"
- board text added: "T-MOS1 Current None/Limit"
- board text added: "T-MOS2 Current None/Limit"
- board text added: "T-Mos1_Drive"
- board text added: "T-Mos2_Drive"
- board text added: "T-PWM/ANALOG"
- board text added: "T-Tot_Current"
- board text added: "VBUS"
- board text added: "VExt"
- board text added: "VOLTAGE GENERATOR"

Commit message: pdf updates
Parts:
- moved C50 574.1 mm to (441.3, 239.5)
- moved C51 574.1 mm to (586.8, 224.8)
- moved C52 574.1 mm to (655.2, 246.8)
- moved R191 574.1 mm to (484.8, 240.2)
- moved R192 574.1 mm to (480.8, 240.2)
- moved R193 574.1 mm to (476.7, 240.2)
- moved R196 574.1 mm to (581.2, 266.0)
- moved R197 574.1 mm to (460.5, 240.2)
- moved R198 574.1 mm to (456.4, 240.2)
- moved R199 574.1 mm to (452.4, 240.2)
- moved R200 574.1 mm to (563.8, 266.0)
- moved R201 574.1 mm to (576.8, 255.5)
- moved R202 574.1 mm to (554.8, 255.5)
- moved R203 574.1 mm to (581.2, 251.1)
- moved R204 574.1 mm to (563.8, 243.5)
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
Commit message: updates
Parts:
- removed the J31 at (27.8, 68.8)
- removed the J36 at (675.8, 190.7)
- removed the R171 at (574.3, 49.0)
- removed the R172 at (564.8, 18.0)
- removed R193: 470K, Resistor_THT:R_Axial_DIN0207_L6.3mm_D2.5mm_P7.62mm_Horizontal
- removed the R194 at (450.5, 268.6)
- removed the R195 at (590.7, 284.5)
- removed the R200 at (563.8, 266.0)
- removed the R202 at (554.8, 255.5)
- removed the R204 at (563.8, 243.5)
- removed the R208 at (663.9, 242.9)
- removed the R210 at (692.2, 253.7)
- removed the R212 at (641.8, 286.5)
- added J55: Conn_01x02_Pin, Connector_Phoenix_GMSTB:PhoenixContact_GMSTBA_2,5_2-G_1x02_P7.50mm_Horizontal, F.Cu at (27.5, 79.0)
- added J56: Conn_01x01_Pin, Connector_PinHeader_2.54mm:PinHeader_1x01_P2.54mm_Vertical, F.Cu at (583.5, 123.5)
- added J57: Conn_01x01_Pin, Connector_PinHeader_2.54mm:PinHeader_1x01_P2.54mm_Vertical, F.Cu at (605.0, 123.5)
- added J58: Conn_01x01_Pin, Connector_PinHeader_2.54mm:PinHeader_1x01_P2.54mm_Vertical, F.Cu at (576.5, 86.8)
- added J59: Conn_01x01_Pin, Connector_PinHeader_2.54mm:PinHeader_1x01_P2.54mm_Vertical, F.Cu at (599.0, 86.8)
- added J60: Conn_01x01_Pin, Connector_PinHeader_2.54mm:PinHeader_1x01_P2.54mm_Vertical, F.Cu at (524.8, 123.5)
- added J61: Conn_01x01_Pin, Connector_PinHeader_2.54mm:PinHeader_1x01_P2.54mm_Vertical, F.Cu at (548.0, 123.5)
- added J62: Conn_01x01_Pin, Connector_PinHeader_2.54mm:PinHeader_1x01_P2.54mm_Vertical, F.Cu at (519.8, 86.5)
- added J63: Conn_01x01_Pin, Connector_PinHeader_2.54mm:PinHeader_1x01_P2.54mm_Vertical, F.Cu at (541.8, 86.8)
- added J64: Conn_01x01_Pin, Connector_PinHeader_2.54mm:PinHeader_1x01_P2.54mm_Vertical, F.Cu at (469.8, 123.5)
- added J65: Conn_01x01_Pin, Connector_PinHeader_2.54mm:PinHeader_1x01_P2.54mm_Vertical, F.Cu at (493.0, 123.5)
- added J66: Conn_01x01_Pin, Connector_PinHeader_2.54mm:PinHeader_1x01_P2.54mm_Vertical, F.Cu at (486.8, 86.2)
- added J67: Conn_01x01_Pin, Connector_PinHeader_2.54mm:PinHeader_1x01_P2.54mm_Vertical, F.Cu at (464.8, 86.2)
- added JP23: SolderJumper_2_Bridged, Jumper:SolderJumper-2_P1.3mm_Bridged2Bar_RoundedPad1.0x1.5mm, F.Cu at (235.5, 124.8)
- added JP24: SolderJumper_2_Bridged, Jumper:SolderJumper-2_P1.3mm_Bridged2Bar_RoundedPad1.0x1.5mm, F.Cu at (239.2, 124.8)
- added TP77: TestPoint_Alt, TestPoint:TestPoint_Loop_D1.80mm_Drill1.0mm_Beaded, F.Cu at (446.8, 182.8)
- added TP78: TestPoint_Alt, TestPoint:TestPoint_Loop_D1.80mm_Drill1.0mm_Beaded, F.Cu at (625.5, 197.0)
- C1, C2, C4: value 1nF -> 100pF
- J19, J27, J32, J37, J38, J39: footprint Connector_Phoenix_GMSTB:PhoenixContact_GMSTBVA_2,5_2-G_1x02_P7.50mm_Vertical -> Connector_Phoenix_GMSTB:PhoenixContact_GMSTBA_2,5_2-G_1x02_P7.50mm_Horizontal
- moved J34 269.2 mm to (615.0, 25.5)
- moved C50 256.2 mm to (594.9, 34.4), turned to 180 degrees
- moved TP70 248.3 mm to (600.7, 43.2), turned to 0 degrees
- moved R197 235.8 mm to (596.2, 47.4)
- moved R192 232.5 mm to (596.2, 38.4), turned to 180 degrees
- moved R198 229.1 mm to (596.2, 58.6)
- moved R191 226.1 mm to (596.2, 43.4), turned to 180 degrees
- moved TP72 224.0 mm to (656.5, 43.2), turned to 0 degrees
- moved R199 222.8 mm to (591.6, 66.2), turned to 180 degrees
- moved R227 222.4 mm to (616.1, 211.3), turned to 90 degrees
- moved R214 216.5 mm to (652.1, 38.5), turned to 180 degrees
- moved R171 215.7 mm to (470.8, 49.0), turned to 180 degrees
- moved C52 212.4 mm to (650.8, 34.5), turned to 180 degrees
- moved R213 212.1 mm to (652.1, 43.5), turned to 180 degrees
- moved R228 211.9 mm to (635.0, 211.3)
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Connections:
- J36 pad 1: GND2 -> +3.3VA
- J36 pad 2: R1_Fire -> T2_Fire
- J36 pad 3: R2_Fire -> T1_Fire
- J36 pad 4: S1_Fire -> S2_Fire
- J36 pad 5: S2_Fire -> S1_Fire
- J36 pad 6: T1_Fire -> R2_Fire
- J36 pad 7: T2_Fire -> R1_Fire
- J36 pad 8: +3.3VA -> GND2
Routing:
- net GND2: track 1226.2 -> 1606.9 mm, vias 14 -> 38
- net +3.3VA: track 123.0 -> 356.1 mm, vias 4 -> 8
- net R_Sec_b: track 69.6 -> 201.2 mm
- net R1_Fire: track 0.00 -> 116.7 mm
- net R2_Fire: track 0.00 -> 101.3 mm
- net S1_Fire: track 0.00 -> 83.9 mm
- net S_Sec_b: track 136.2 -> 211.7 mm
- net T_OptoTriac: track 71.3 -> 6.29 mm
- net S2_Fire: track 0.00 -> 60.5 mm
- net Notr: track 117.9 -> 173.4 mm
- net T_Sec_b: track 112.4 -> 164.6 mm
- net T1_Fire: track 0.00 -> 43.6 mm
- net Net-(J31-Pin_1): track 77.8 -> 120.7 mm
- net T2_Fire: track 0.00 -> 41.1 mm
- net T_Phase_Volt: track 0.00 -> 38.5 mm
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- added copper zone on B.Cu, net GND2
- added copper zone on B.Cu, net GNDPWR
Other:
- board size 656.3 x 217.1 mm -> 644.3 x 199.1 mm
- board text added: "12V LED"
- board text added: "3V3 LED"
- board text added: "CT_R1_Inp"
- board text added: "CT_R1_Out"
- board text added: "CT_R2_Inp"
- board text added: "CT_R2_Out"
- board text added: "CT_S1_Inp"
- board text added: "CT_S1_Out"
- board text added: "CT_S2_Inp"
- board text added: "CT_S2_Out"
- board text added: "CT_T1_Inp"
- board text added: "CT_T1_Out"
- board text added: "CT_T2_Inp"
- board text added: "CT_T2_Out"
- board text added: "GND POWER"
- board text added: "PCB Copper : 70um 2 layers"
- board text added: "R Grid Volt"
- board text added: "R Opto Out"
- board text added: "R1"
- board text added: "R1 Fire"
- board text added: "R1 G-K"
- board text added: "R2"
- board text added: "R2 Fire"
- board text added: "R2 G-K"
- board text added: "S Grid Volt"
- board text added: "S Opto Out"
- board text added: "S1"
- board text added: "S1 Fire"
- board text added: "S1 G-K"
- board text added: "S2"
- board text added: "S2 Fire"
- board text added: "S2 G-K"
- board text added: "T Grid Volt"
- board text added: "T Opto Out"
- board text added: "T1"
- board text added: "T1 Fire"
- board text added: "T1 G-K"
- board text added: "T2"
- board text added: "T2 Fire"
- board text added: "T2 G-K"
- board text added: "VDD"
- board text added: "VDD LED"
- board text removed: "PCB Dimensions : 384x246 mm Copper : 70um 2 layers X: 19,5 - 403,5 Y: 17,5 - 263,5"

Commit message: updates2
Parts:
- moved R119 10.1 mm to (494.8, 170.2)
- moved TP10 8.12 mm to (292.9, 156.1)
- moved R139 6.42 mm to (542.2, 170.2), turned to 0 degrees
- moved R46 5.87 mm to (303.0, 157.5)
- moved R35 3.78 mm to (68.4, 146.5)
- moved R74 2.46 mm to (266.2, 146.5)
- moved R86 2.46 mm to (266.2, 144.2)
- moved R87 2.16 mm to (267.2, 155.0), turned to 180 degrees
- moved R40 2.03 mm to (306.8, 153.0), turned to 180 degrees
- moved R26 1.69 mm to (68.5, 143.5)
- moved R88 1.51 mm to (266.2, 157.5)
- moved R91 1.12 mm to (266.2, 149.2)
- moved C35 1.09 mm to (537.5, 176.8), turned to 0 degrees
- moved R61 0.96 mm to (77.6, 131.4)
- moved TP1 0.95 mm to (81.7, 129.3)
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Routing:
- net GND: track 925.0 -> 853.2 mm, vias 53 -> 65
- net Net-(R43-Pad1): track 16.3 -> 39.5 mm
- net T_Mos_I_2: track 67.4 -> 90.5 mm
- net Net-(R29-Pad1): track 14.6 -> 34.9 mm
- net GND2: track 1606.9 -> 1626.2 mm, vias 38 -> 61
- net Net-(C30-Pad2): track 63.0 -> 82.0 mm, vias 3 -> 4
- net +3.3V: track 439.8 -> 457.9 mm, vias 2 -> 8
- net T_Mos_I_1: track 111.2 -> 127.4 mm
- net Net-(C4-Pad1): track 0.00 -> 15.7 mm
- net Net-(U3D-+): track 0.00 -> 11.9 mm
- net Net-(U1D--): track 0.00 -> 10.7 mm
- net Net-(C25-Pad2): track 0.00 -> 10.2 mm
- net T_MosD_2: track 26.0 -> 35.8 mm, vias 0 -> 4
- net Net-(R122-Pad1): track 29.3 -> 37.6 mm
- net Net-(U3D--): track 0.00 -> 8.10 mm
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Other:
- board text added: "R_High Analog_Gain"
- board text added: "R_High_Adj"
- board text added: "R_High_Analog"
- board text added: "R_High_Mosfet"
- board text added: "R_High_PWM"
- board text added: "R_Low Analog_Gain"
- board text added: "R_Low_Adj"
- board text added: "R_Low_Analog"
- board text added: "R_Low_Mosfet"
- board text added: "R_Low_PWM"
- board text added: "S_High_Analog"
- board text added: "S_High_Analog_Gain"
- board text added: "S_High_PWM"
- board text added: "S_Low_Analog"
- board text added: "S_Low_PWM"
- board text added: "T_High_Analog"
- board text added: "T_High_Mosfet"
- board text added: "T_High_PWM"
- board text added: "T_Low_Analog"
- board text added: "T_Low_PWM"
