File: Cur_Emul/Cur_Emul.kicad_pcb (KiCad board)
At the start: 2 copper layers, 644.3 x 199.1 mm, 521 parts, among them J1 Screw_Terminal_01x01, J10 Screw_Terminal_01x01, J11 Screw_Terminal_01x01, J12 Screw_Terminal_01x01, J13 Screw_Terminal_01x01, J14 Screw_Terminal_01x01, J15 Screw_Terminal_01x01, J16 Screw_Terminal_01x01, J17 Conn_01x04_Pin, J18 Conn_01x02_Pin, J19 Conn_01x02_Pin, J2 Screw_Terminal_01x01, J20 Conn_01x04_Pin, J21 Screw_Terminal_01x01, J22 Screw_Terminal_01x01, J23 Conn_01x06_Pin, J24 Conn_01x08_Pin, J25 Conn_01x08_Pin, J26 Conn_01x04_Pin, J27 Conn_01x02_Pin, J28 Conn_01x04_Pin, J29 Conn_01x02_Pin, J3 Screw_Terminal_01x01, J30 Conn_01x02_Pin, J31 Conn_01x02_Pin, J32 Conn_01x02_Pin, J33 Conn_01x08_Pin, J34 Conn_01x06_Pin, J35 Conn_01x04_Pin, J36 Conn_01x08_Pin, J37 Conn_01x02_Pin, J38 Conn_01x02_Pin, J39 Conn_01x02_Pin, J4 Screw_Terminal_01x01, J40 Conn_01x01_Pin, J41 Conn_01x01_Pin, J42 Conn_01x01_Pin, J43 Conn_01x01_Pin, J44 Conn_01x01_Pin, J45 Conn_01x01_Pin, J46 Conn_01x01_Pin, J47 Conn_01x01_Pin, J48 Conn_01x01_Pin, J49 Conn_01x04_Pin, J5 Screw_Terminal_01x01, J50 Conn_01x04_Pin, J51 Conn_01x02_Pin, J52 Conn_01x02_Pin, J53 Conn_01x02_Pin, J54 Conn_01x02_Pin, J55 Conn_01x02_Pin, J56 Conn_01x01_Pin, J57 Conn_01x01_Pin, J58 Conn_01x01_Pin, J59 Conn_01x01_Pin, J6 Screw_Terminal_01x01, J60 Conn_01x01_Pin, J61 Conn_01x01_Pin, J62 Conn_01x01_Pin, J63 Conn_01x01_Pin, J64 Conn_01x01_Pin, J65 Conn_01x01_Pin, J66 Conn_01x01_Pin, J67 Conn_01x01_Pin, J7 Screw_Terminal_01x01, J8 Screw_Terminal_01x01, J9 Screw_Terminal_01x01, M1 IXTH64N10L2, M10 IRF530, M11 IRF530, M12 IRF530, M2 IXTH64N10L2, M3 IXTH64N10L2, M4 IXTH64N10L2, M5 IXTH64N10L2, M6 IXTH64N10L2, M7 IRF530, M8 IRF530, M9 IRF530, T1 Transformer_1P_2S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

Commit message: updates3
Parts:
- moved R93 4.83 mm to (204.4, 162.6)
- moved R31 3.38 mm to (185.5, 163.1)
- moved R37 2.70 mm to (185.5, 160.1)
- moved TP8 2.69 mm to (200.4, 143.8)
- moved JP6 1.29 mm to (201.5, 159.7)
- moved R69 0.34 mm to (195.5, 146.7)
- moved R67 0.28 mm to (199.7, 146.8)
- moved JP2 0.27 mm to (182.2, 147.1)
- moved R38 0.20 mm to (183.3, 144.6)
- moved R71 0.20 mm to (199.8, 152.0), turned to 180 degrees
- moved R32 0.15 mm to (183.0, 150.0)
Routing:
- net S_Mos_I_2: track 71.6 -> 123.7 mm
- net Net-(R34-Pad2): track 0.00 -> 34.5 mm
- net S_MosD_2: track 136.3 -> 167.6 mm
- net S_Mos_I_1: track 158.5 -> 186.2 mm
- net GND: track 853.2 -> 826.6 mm, vias 65 -> 80
- net Net-(R31-Pad1): track 0.00 -> 11.9 mm, vias 0 -> 2
- net Net-(U2D-+): track 0.00 -> 11.3 mm
- net Net-(JP6-C): track 6.29 -> 17.3 mm
- net Net-(U2D--): track 2.50 -> 13.3 mm
- net Net-(C8-Pad2): track 0.00 -> 9.47 mm
- net Net-(U2C--): track 1.88 -> 10.5 mm
- net R_PWM_Analog: track 175.5 -> 182.4 mm
- net Net-(JP4-C): track 0.00 -> 6.30 mm
- net Net-(JP2-C): track 0.00 -> 5.98 mm
- net Net-(JP4-A): track 0.00 -> 5.30 mm
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Other:
- outline, holes or cut-outs redrawn

Commit message: updates4
Parts:
- added C54: 1nF, Capacitor_SMD:C_0805_2012Metric_Pad1.18x1.45mm_HandSolder, F.Cu at (312.2, 159.3)
- added C55: 1nF, Capacitor_SMD:C_0805_2012Metric_Pad1.18x1.45mm_HandSolder, F.Cu at (191.9, 164.0)
- added C56: 1nF, Capacitor_SMD:C_0805_2012Metric_Pad1.18x1.45mm_HandSolder, F.Cu at (73.7, 149.5)
- C9: value 300uF -> 300uF / 50V
- R10, R11, R12, R14, R15, R16, R18, R19, R20, R22, R23, R24, R3, R4, R6, R7, R8: value R -> 10mR
- R158, R44, R48: value R -> 4R7; footprint Resistor_THT:R_Axial_DIN0204_L3.6mm_D1.6mm_P7.62mm_Horizontal -> Resistor_THT:R_Axial_DIN0411_L9.9mm_D3.6mm_P12.70mm_Horizontal
- R159, R160, R47: value R -> 4R7; footprint Resistor_SMD:R_Shunt_Vishay_WSR2_WSR3 -> Resistor_THT:R_Axial_DIN0411_L9.9mm_D3.6mm_P12.70mm_Horizontal
- R2: value 3 X 0.001R -> 10mR
- R68: value R -> 1R
- moved R159 46.1 mm to (501.3, 109.5)
- moved R160 41.9 mm to (563.9, 110.3)
- moved R47 41.0 mm to (454.2, 109.7)
- moved R48 39.1 mm to (558.2, 110.2)
- moved TP17 38.9 mm to (539.4, 157.1)
- moved R44 38.9 mm to (447.6, 109.6)
- moved R158 34.3 mm to (507.9, 109.7)
- moved D2 24.3 mm to (450.2, 88.4)
- moved R164 19.7 mm to (447.2, 88.3)
- moved R161 19.2 mm to (447.2, 84.3)
- moved TP50 8.50 mm to (518.7, 158.8)
- moved R31 3.48 mm to (185.3, 166.6)
- moved TP69 3.14 mm to (450.1, 93.5)
- moved TP2 2.98 mm to (64.4, 119.0)
- moved R80 2.84 mm to (220.3, 161.5)
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Routing:
- net GND2: track 1626.2 -> 1745.5 mm, vias 61 -> 69
- net S_Volt_Lim: track 77.3 -> 117.5 mm
- net +12VA: track 344.3 -> 371.0 mm
- net +15V: track 414.3 -> 439.5 mm
- net T_Volt_Lim: track 82.0 -> 105.3 mm
- net R_Volt_Lim: track 73.7 -> 94.0 mm
- net +3.3VA: track 362.9 -> 381.6 mm
- net VDD: track 312.2 -> 298.2 mm
- net R_Volt_MosH: track 48.7 -> 61.0 mm
- net S_Sec_b: track 211.7 -> 202.7 mm
- net T_Sec_a: track 146.3 -> 137.8 mm
- net R_Mos_I_1: track 148.6 -> 141.5 mm
- net VBUS: track 1149.8 -> 1155.5 mm, vias 5 -> 4
- net R_Mos_I_2: track 144.2 -> 149.8 mm
- net T_MosD_2: track 35.8 -> 40.6 mm
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Other:
- outline, holes or cut-outs redrawn
- board text added: "R_H_Gain"
- board text added: "R_L_Gain"
- board text added: "S_H_Gain"
- board text added: "S_High_Mosfet"
- board text added: "S_L_Gain"
- board text added: "S_Low Analog_Gain"
- board text added: "S_Low_Mosfet"
- board text added: "T_H_Gain"
- board text added: "T_High_Analog_Gain"
- board text added: "T_L_Gain"
- board text added: "T_Low_Analog_Gain"
- board text added: "T_Low_Mosfet"
- board text removed: "3V3 Input Bus/Ext"
- board text removed: "Input.1"
- board text removed: "Input.2"
- board text removed: "Input.3"
- board text removed: "R_High_Adj"
- board text removed: "R_Low_Adj"

Commit message: updates4
Other:
- board text added: "ABB EMULATOR"
- board text added: "Current Generator 384x 166 mm 70um 2 layers"
- board text added: "Voltage Generator 237 x 194 mm 35um 2 layers"
- board text removed: "PCB Copper : 70um 2 layers"
Changed lines of the file:
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@@
 		(pcbplotparams
 			(layerselection 0x00000000_00000000_55555555_5755f5ff)
-			(plot_on_all_layers_selection 0x00000000_00000000_00000000_00000000)
+			(plot_on_all_layers_selection 0x00000000_00000000_00000000_020020ae)
 			(disableapertmacros no)
 			(usegerberextensions no)
@@
 			(drillshape 0)
 			(scaleselection 1)
-			(outputdirectory "")
+			(outputdirectory "GERBER/")
 		)
 	)
@@
 	)
 	(gr_text "CURRENT GENERATOR"
-		(at 342.5 26.25 0)
+		(at 345.2 31.2 0)
 		(layer "F.SilkS")
 		(effects
@@
 		)
 	)
-	(gr_text "EMULATOR"
-		(at 219.202 31.75 0)
+	(gr_text "ABB EMULATOR"
+		(at 352.8 25.1 0)
 		(layer "F.SilkS")
 		(effects
@@
 	)
 	(gr_text "VOLTAGE GENERATOR"
-		(at 544.97 29.85 0)
+		(at 538.3 34.1 0)
 		(layer "F.SilkS")
 		(effects
@@
 		)
 	)
+	(gr_text "ABB EMULATOR"
+		(at 546.1 29.3 0)
+		(layer "F.SilkS")
+		(effects
+			(font
+				(size 3 3)
+				(thickness 0.3)
+				(bold yes)
+			)
+			(justify left bottom)
+		)
+	)
 	(gr_text "T-MOS2 Current\n  None/Limit"
 		(at 283.6 150.4 0)
@@
 		)
 	)
+	(gr_text "Voltage Generator\n237 x 194 mm\n35um 2 layers"
+		(at 365.1 213.8 0)
+		(layer "F.SilkS")
+		(effects
+			(font
+				(size 2 2)
+				(thickness 0.1)
+			)
+			(justify left bottom)
+		)
+	)
 	(gr_text "Star"
 		(at 508.25 64.25 0)
@@
 		)
 	)
-	(gr_text "PCB Copper :  70um 2 layers\n"
-		(at 349 192.25 0)
+	(gr_text "Current Generator\n384x 166 mm\n70um 2 layers"
+		(at 365 194.9 0)
 		(layer "F.SilkS")
 		(effects
@@
 		(min_thickness 0.25)
 		(filled_areas_thickness no)
-		(fill
+		(fill yes
 			(thermal_gap 0.5)
 			(thermal_bridge_width 0.5)
@@
 		(min_thickness 0.25)
 		(filled_areas_thickness no)
-		(fill
+		(fill yes
 			(thermal_gap 0.5)
 			(thermal_bridge_width 0.5)
@@
 		(min_thickness 0.25)
 		(filled_areas_thickness no)
-		(fill
+		(fill yes
 			(thermal_gap 0.5)
 			(thermal_bridge_width 0.5)
@@
 		(min_thickness 0.25)
 		(filled_areas_thickness no)
-		(fill
+		(fill yes
 			(thermal_gap 0.5)
 			(thermal_bridge_width 0.5)
@@
 		(min_thickness 0.25)
 		(filled_areas_thickness no)
-		(fill
+		(fill yes
 			(thermal_gap 0.5)
 			(thermal_bridge_width 0.5)
@@
 		(min_thickness 0.25)
 		(filled_areas_thickness no)
-		(fill
+		(fill yes
 			(thermal_gap 0.5)
 			(thermal_bridge_width 0.5)
@@
 		(min_thickness 0.25)
 		(filled_areas_thickness no)
-		(fill
+		(fill yes
 			(thermal_gap 0.5)
 			(thermal_bridge_width 0.5)
@@
 		(min_thickness 0.25)
 		(filled_areas_thickness no)
-		(fill
+		(fill yes
 			(thermal_gap 0.5)
 			(thermal_bridge_width 0.5)
@@
 		(min_thickness 0.25)
 		(filled_areas_thickness no)
-		(fill
+		(fill yes
 			(thermal_gap 0.5)
 			(thermal_bridge_width 0.5)
@@
 		(min_thickness 0.25)
 		(filled_areas_thickness no)
-		(fill
+		(fill yes
 			(thermal_gap 0.5)
 			(thermal_bridge_width 0.5)
@@
 		(min_thickness 0.25)
 		(filled_areas_thickness no)
-		(fill
+		(fill yes
 			(thermal_gap 0.5)
 			(thermal_bridge_width 0.5)
@@
 		(min_thickness 0.25)
 		(filled_areas_thickness no)
-		(fill
+		(fill yes
 			(thermal_gap 0.5)
 			(thermal_bridge_width 0.5)
@@
 		(min_thickness 0.25)
 		(filled_areas_thickness no)
-		(fill
+		(fill yes
 			(thermal_gap 0.5)
 			(thermal_bridge_width 0.5)
