File: Cur_Emul/Cur_Emul.kicad_pcb (KiCad board)
At the start: 2 copper layers, 644.3 x 199.1 mm, 524 parts, among them J1 Screw_Terminal_01x01, J10 Screw_Terminal_01x01, J11 Screw_Terminal_01x01, J12 Screw_Terminal_01x01, J13 Screw_Terminal_01x01, J14 Screw_Terminal_01x01, J15 Screw_Terminal_01x01, J16 Screw_Terminal_01x01, J17 Conn_01x04_Pin, J18 Conn_01x02_Pin, J19 Conn_01x02_Pin, J2 Screw_Terminal_01x01, J20 Conn_01x04_Pin, J21 Screw_Terminal_01x01, J22 Screw_Terminal_01x01, J23 Conn_01x06_Pin, J24 Conn_01x08_Pin, J25 Conn_01x08_Pin, J26 Conn_01x04_Pin, J27 Conn_01x02_Pin, J28 Conn_01x04_Pin, J29 Conn_01x02_Pin, J3 Screw_Terminal_01x01, J30 Conn_01x02_Pin, J31 Conn_01x02_Pin, J32 Conn_01x02_Pin, J33 Conn_01x08_Pin, J34 Conn_01x06_Pin, J35 Conn_01x04_Pin, J36 Conn_01x08_Pin, J37 Conn_01x02_Pin, J38 Conn_01x02_Pin, J39 Conn_01x02_Pin, J4 Screw_Terminal_01x01, J40 Conn_01x01_Pin, J41 Conn_01x01_Pin, J42 Conn_01x01_Pin, J43 Conn_01x01_Pin, J44 Conn_01x01_Pin, J45 Conn_01x01_Pin, J46 Conn_01x01_Pin, J47 Conn_01x01_Pin, J48 Conn_01x01_Pin, J49 Conn_01x04_Pin, J5 Screw_Terminal_01x01, J50 Conn_01x04_Pin, J51 Conn_01x02_Pin, J52 Conn_01x02_Pin, J53 Conn_01x02_Pin, J54 Conn_01x02_Pin, J55 Conn_01x02_Pin, J56 Conn_01x01_Pin, J57 Conn_01x01_Pin, J58 Conn_01x01_Pin, J59 Conn_01x01_Pin, J6 Screw_Terminal_01x01, J60 Conn_01x01_Pin, J61 Conn_01x01_Pin, J62 Conn_01x01_Pin, J63 Conn_01x01_Pin, J64 Conn_01x01_Pin, J65 Conn_01x01_Pin, J66 Conn_01x01_Pin, J67 Conn_01x01_Pin, J7 Screw_Terminal_01x01, J8 Screw_Terminal_01x01, J9 Screw_Terminal_01x01, M1 IXTH64N10L2, M10 IRF530, M11 IRF530, M12 IRF530, M2 IXTH64N10L2, M3 IXTH64N10L2, M4 IXTH64N10L2, M5 IXTH64N10L2, M6 IXTH64N10L2, M7 IRF530, M8 IRF530, M9 IRF530, T1 Transformer_1P_2S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

Commit message: with Fabr. Outputs
Parts:
- removed C1, C2, C4: 100pF, Capacitor_SMD:C_0805_2012Metric_Pad1.18x1.45mm_HandSolder
- removed J49, J50: Conn_01x04_Pin, Connector_Phoenix_GMSTB:PhoenixContact_GMSTBA_2,5_4-G-7,62_1x04_P7.62mm_Horizontal
- removed R100, R122, R123, R142, R143, R29, R34, R43, R51: 100R, Resistor_SMD:R_0805_2012Metric_Pad1.20x1.40mm_HandSolder
- removed R171, R194, R224: 220R, Resistor_THT:R_Axial_DIN0207_L6.3mm_D2.5mm_P7.62mm_Horizontal
- added D24: 1N5407, Diode_THT:D_DO-201AD_P15.24mm_Horizontal, F.Cu at (432.3, 134.8)
- added D25: 1N5407, Diode_THT:D_DO-201AD_P15.24mm_Horizontal, F.Cu at (48.0, 147.5)
- added D26: 1N5407, Diode_THT:D_DO-201AD_P15.24mm_Horizontal, F.Cu at (24.7, 109.1)
- added Fiducial: Fiducial_1.5mm_Mask3mm, Fiducial:Fiducial_1.5mm_Mask3mm, F.Cu at (643.3, 198.5)
- added Fiducial: Fiducial_1.5mm_Mask3mm, Fiducial:Fiducial_1.5mm_Mask3mm, F.Cu at (465.3, 66.5)
- added Fiducial: Fiducial_1.5mm_Mask3mm, Fiducial:Fiducial_1.5mm_Mask3mm, F.Cu at (389.9, 42.0)
- added Fiducial: Fiducial_1.5mm_Mask3mm, Fiducial:Fiducial_1.5mm_Mask3mm, F.Cu at (374.6, 177.6)
- added Fiducial: Fiducial_1.5mm_Mask3mm, Fiducial:Fiducial_1.5mm_Mask3mm, F.Cu at (636.9, 56.6)
- added Fiducial: Fiducial_1.5mm_Mask3mm, Fiducial:Fiducial_1.5mm_Mask3mm, F.Cu at (454.2, 213.6)
- added Fiducial: Fiducial_1.5mm_Mask3mm, Fiducial:Fiducial_1.5mm_Mask3mm, F.Cu at (75.4, 175.8)
- added Fiducial: Fiducial_1.5mm_Mask3mm, Fiducial:Fiducial_1.5mm_Mask3mm, F.Cu at (38.9, 28.5)
- added G***: LOGO, Emul_footprint:ABB_Logo2, F.Cu at (626.6, 87.7)
- added G***: LOGO, Emul_footprint:ABB_Logo2, F.Cu at (583.7, 175.6)
- added G***: LOGO, Emul_footprint:ABB_Logo2, F.Cu at (365.4, 141.2)
- added G***: LOGO, Emul_footprint:Ilker_logo4, F.Cu at (508.6, 187.0)
- added G***: LOGO, Emul_footprint:ABB_Logo2, F.Cu at (237.3, 32.1)
- added G***: LOGO, Emul_footprint:Ilker_logo4, F.Cu at (123.9, 139.5)
- added J68: 2x7.50mm_Vertical_PhoenixContact_GMSTB, Connector_Phoenix_GMSTB:PhoenixContact_GMSTBVA_2,5_2-G_1x02_P7.50mm_Vertical, F.Cu at (552.5, 46.4)
- added J69: 2x7.50mm_Vertical_PhoenixContact_GMSTB, Connector_Phoenix_GMSTB:PhoenixContact_GMSTBVA_2,5_2-G_1x02_P7.50mm_Vertical, F.Cu at (507.1, 48.6)
- added J70: 2x7.50mm_Vertical_PhoenixContact_GMSTB, Connector_Phoenix_GMSTB:PhoenixContact_GMSTBVA_2,5_2-G_1x02_P7.50mm_Vertical, F.Cu at (456.6, 52.4)
- added J72: 2x7.50mm_Horizontal_PhoenixContact_GMSTBA, Connector_Phoenix_GMSTB:PhoenixContact_GMSTBA_2,5_2-G_1x02_P7.50mm_Horizontal, F.Cu at (35.1, 171.4)
- added J73: 2x7.50mm_Horizontal_PhoenixContact_GMSTBA, Connector_Phoenix_GMSTB:PhoenixContact_GMSTBA_2,5_2-G_1x02_P7.50mm_Horizontal, F.Cu at (51.2, 171.4)
- added J80: 2x7.50mm_Horizontal_PhoenixContact_GMSTBA, Connector_Phoenix_GMSTB:PhoenixContact_GMSTBA_2,5_2-G_1x02_P7.50mm_Horizontal, F.Cu at (439.4, 186.1)
- added J81: 2x7.50mm_Horizontal_PhoenixContact_GMSTBA, Connector_Phoenix_GMSTB:PhoenixContact_GMSTBA_2,5_2-G_1x02_P7.50mm_Horizontal, F.Cu at (439.4, 202.2)
- C10, C49: value 1uF MKT -> 1uF/50V MKT
- C11, C12, C13, C14, C19, C20, C37, C38, C39, C40, C45: value C_Polarized -> 10uF/50V
- C15, C16, C17, C18, C22, C23, C41, C42, C43, C44, C46: value C_Polarized -> 10nF/50V
- C21, C24, C26, C27, C28, C29, C30, C33, C34: value 1uF -> 1uF/50V
- C25, C7, C8: value 10pF -> 10nF/50V
- C3, C47: value C_Polarized -> 100uF/50V
- C31, C32, C35, C36, C5, C54, C55, C56, C6: value 1nF -> 10nF/50V
- C48: value C_Polarized -> 1000uF/50V
- C50, C51, C52: value 100nF -> 100nF/50V
- C9: value 300uF / 50V -> 300uF/50V
- J1, J10, J11, J12, J13, J14, J15, J16, J2, J21, J22, J3, J4, J5, J6, J7, J8, J9: value Screw_Terminal_01x01 -> Wuerth_REDCUBE-74651175_ScrewTerminal
- J17, J26, J28: value Conn_01x04_Pin -> Conn_01x04_Pin_JST_2.5mm
- J18, J29, J30: value Conn_01x02_Pin -> 2x7.50mm_Vertical_PhoenixContact_GMSTB
- J19, J27, J31, J32, J37, J38, J39, J51, J52, J53, J54, J55: value Conn_01x02_Pin -> 2x7.50mm_Horizontal_PhoenixContact_GMSTBA
- J20, J35: value Conn_01x04_Pin -> Conn_01x04_Pin_JST_2.0mm
- J23, J34: value Conn_01x06_Pin -> Conn_01x06_Pin_JST_2.0mm
- J24, J25, J33, J36: value Conn_01x08_Pin -> Conn_01x08_Pin_JST_2.0mm
- J40, J41, J42, J43, J44, J45, J46, J47, J48, J56, J57, J58, J59, J60, J61, J62, J63, J64, J65, J66, J67: value Conn_01x01_Pin -> PinHeader_1x2.54mm
- R10, R11, R12, R14, R15, R16, R18, R19, R2, R20, R22, R23, R24, R3, R4, R6, R7, R8: value 10mR -> 10mOhm_Vishay_WSR3_Shunt
- R154: value 1K22 -> 1K22 / %1
- R155: value 110R -> 110R / %1
- R156: value 450R -> 450R / %1
- R157: value 750R -> 750R / %1
- R158, R159, R160, R44, R47, R48: value 4R7 -> 4R7/2W
- R167, R169, R208: value 10K -> 100R
- R168, R170, R210: value 10K -> 100K
- R172, R195, R212: value 220R -> 100K
- R173, R174, R175: footprint Resistor_SMD:R_0805_2012Metric_Pad1.20x1.40mm_HandSolder -> Resistor_THT:R_Axial_DIN0207_L6.3mm_D2.5mm_P7.62mm_Horizontal
- R68: value 1R -> 1R/100W
- RV1, RV2, RV3, RV4, RV5, RV6, RV7, RV8, RV9: value 10K -> 10K_SMD_Pot
- TP1, TP10, TP11, TP12, TP13, TP14, TP15, TP16, TP17, TP18, TP19, TP2, TP20, TP27, TP28, TP29, TP3, TP30, TP31, TP32, TP33, TP34, TP35, TP36, TP37, TP38, TP4, TP41, TP42, TP43, TP44, TP45, TP46, TP47, TP48, TP49, TP5, TP50, TP51, TP52, TP53, TP54, TP55, TP56, TP57, TP58, TP59, TP6, TP60, TP61, TP62, TP63, TP64, TP65, TP66, TP67, TP68, TP69, TP7, TP70, TP71, TP72, TP73, TP74, TP75, TP76, TP77, TP78, TP8, TP9: value TestPoint_Alt -> Test_Point_THT_KeyStone
- TP21, TP22, TP23, TP24, TP25, TP26, TP39, TP40: value TestPoint -> Test_Pad_Not_A_Component
- U1, U10, U11, U12, U2, U4, U8, U9: value Opamp_Quad -> Opamp_Quad_OPA_4196
- U14, U16, U18: value TLP3023 -> MOC3023M; footprint Package_DIP:Toshiba_11-7A9 -> Package_DIP:DIP-6_W7.62mm
- U17, U19, U20, U21, U22, U23: value SFH6206-2T -> SFH620A-2; footprint Package_DIP:SMDIP-4_W9.53mm_Clearance8mm -> Package_DIP:DIP-4_W7.62mm
- U3: value Opamp_Quad -> Opamp_Quad_OPA_4196; footprint Library:SOIC-14_3.9x8.7mm_P1.27mm_ilker -> Package_SO:SOIC-14_3.9x8.7mm_P1.27mm
- moved D16 44.5 mm to (80.9, 160.8)
- moved R163 44.5 mm to (84.4, 160.8)
- moved R175 33.7 mm to (559.3, 31.1), turned to 0 degrees
- moved R168 32.7 mm to (440.4, 50.6), turned to 0 degrees
- moved R208 25.3 mm to (571.1, 46.6), turned to 90 degrees
- moved R170 22.5 mm to (488.9, 47.2), turned to 0 degrees
- moved U18 20.2 mm to (554.6, 31.1)
- moved R119 19.2 mm to (497.1, 189.3), turned to 180 degrees
- moved JP21 16.6 mm to (431.1, 114.6), turned to 180 degrees
- moved R212 16.5 mm to (545.3, 40.3)
- moved R169 14.8 mm to (523.5, 48.8), turned to 90 degrees
- moved TP76 14.7 mm to (622.0, 212.8)
- moved R210 14.4 mm to (534.6, 47.3), turned to 0 degrees
- moved TP64 14.4 mm to (622.6, 194.0)
- moved TP62 13.6 mm to (496.5, 30.3)
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Connections:
- C31 pad 1: Net-(C31-Pad1) -> Net-(U10D--)
- C31 pad 2: GND2 -> Net-(C31-Pad2)
- C32 pad 1: Net-(C32-Pad1) -> Net-(U10C--)
- C32 pad 2: GND2 -> Net-(C32-Pad2)
- C35 pad 1: Net-(C35-Pad1) -> Net-(U11D--)
- C35 pad 2: GND2 -> Net-(C35-Pad2)
- C36 pad 1: Net-(C36-Pad1) -> Net-(U11C--)
- C36 pad 2: GND2 -> Net-(C36-Pad2)
- C49 pad 1: Net-(J31-Pin_1) -> Net-(D25-K)
- C5 pad 1: Net-(C5-Pad1) -> Net-(U8C--)
- C5 pad 2: GND2 -> Net-(C5-Pad2)
- C6 pad 1: Net-(C6-Pad1) -> Net-(U8D--)
- C6 pad 2: GND2 -> Net-(C6-Pad2)
- J31 pad 1: Net-(J31-Pin_1) -> Net-(D25-A)
- J34 pad 6: unconnected-(J34-Pin_6-Pad6) -> GND2
- J54 pad 1: Net-(J31-Pin_1) -> VBUS
- J55 pad 1: Net-(J31-Pin_1) -> Net-(D26-A)
- JP11 pad 1: Net-(J31-Pin_1) -> Net-(D25-K)
- JP21 pad 1: Net-(J51-Pin_1) -> Net-(J52-Pin_1)
- JP21 pad 2: Net-(D1-K) -> Net-(D24-A)
- JP21 pad 3: Net-(J52-Pin_1) -> Net-(J51-Pin_1)
- JP22 pad 1: Net-(J31-Pin_1) -> Net-(D25-K)
- R124 pad 1: Net-(C32-Pad1) -> Net-(C32-Pad2)
- R125 pad 1: Net-(C31-Pad1) -> Net-(C31-Pad2)
- R144 pad 1: Net-(C36-Pad1) -> Net-(C36-Pad2)
- R145 pad 1: Net-(C35-Pad1) -> Net-(C35-Pad2)
- R167 pad 1: V1_Line -> R_Sec_b
- R168 pad 1: Net-(R167-Pad2) -> Net-(R168-Pad1)
- R168 pad 2: V1_Motor -> Notr
- R169 pad 1: V2_Line -> S_Sec_b
- R170 pad 1: Net-(R169-Pad2) -> Net-(R170-Pad1)
- R170 pad 2: V2_Motor -> Notr
- R172 pad 1: Net-(R172-Pad1) -> V2_Motor
- R172 pad 2: Notr -> Net-(R170-Pad1)
- R195 pad 1: Net-(R195-Pad1) -> V1_Motor
- R195 pad 2: Notr -> Net-(R168-Pad1)
- R208 pad 1: V3_Line -> T_Sec_b
- R210 pad 1: Net-(R208-Pad2) -> Net-(R210-Pad1)
- R210 pad 2: V3_Motor -> Notr
- R212 pad 1: Net-(R212-Pad1) -> V3_Motor
- R212 pad 2: Notr -> Net-(R210-Pad1)
- R27 pad 1: Net-(C2-Pad1) -> Net-(C56-Pad2)
- R28 pad 1: Net-(C2-Pad1) -> Net-(C56-Pad2)
- R32 pad 1: Net-(C1-Pad1) -> Net-(C55-Pad2)
- R33 pad 1: Net-(C1-Pad1) -> Net-(C55-Pad2)
- R41 pad 1: Net-(C4-Pad1) -> Net-(C54-Pad2)
- R42 pad 1: Net-(C4-Pad1) -> Net-(C54-Pad2)
- R52 pad 1: Net-(C5-Pad1) -> Net-(C5-Pad2)
- R53 pad 1: Net-(C6-Pad1) -> Net-(C6-Pad2)
- RV4 pad 1: Net-(R51-Pad1) -> Net-(C5-Pad2)
- RV4 pad 2: Net-(R51-Pad1) -> Net-(C5-Pad2)
- RV5 pad 1: Net-(R100-Pad1) -> Net-(C6-Pad2)
- RV5 pad 2: Net-(R100-Pad1) -> Net-(C6-Pad2)
- RV6 pad 1: Net-(R122-Pad1) -> Net-(C31-Pad2)
- RV6 pad 2: Net-(R122-Pad1) -> Net-(C31-Pad2)
- RV7 pad 1: Net-(R123-Pad1) -> Net-(C32-Pad2)
- RV7 pad 2: Net-(R123-Pad1) -> Net-(C32-Pad2)
- RV8 pad 1: Net-(R142-Pad1) -> Net-(C35-Pad2)
- RV8 pad 2: Net-(R142-Pad1) -> Net-(C35-Pad2)
- RV9 pad 1: Net-(R143-Pad1) -> Net-(C36-Pad2)
- RV9 pad 2: Net-(R143-Pad1) -> Net-(C36-Pad2)
- TP31 pad 1: Net-(R51-Pad1) -> Net-(C5-Pad2)
- TP34 pad 1: Net-(R100-Pad1) -> Net-(C6-Pad2)
- TP37 pad 1: Net-(J31-Pin_1) -> Net-(D25-K)
- TP47 pad 1: Net-(R122-Pad1) -> Net-(C31-Pad2)
- TP48 pad 1: Net-(R123-Pad1) -> Net-(C32-Pad2)
- TP55 pad 1: Net-(R142-Pad1) -> Net-(C35-Pad2)
- TP56 pad 1: Net-(R143-Pad1) -> Net-(C36-Pad2)
- U10 pad 14: Net-(R122-Pad1) -> Net-(C31-Pad2)
- U10 pad 8: Net-(R123-Pad1) -> Net-(C32-Pad2)
- U11 pad 14: Net-(R142-Pad1) -> Net-(C35-Pad2)
- U11 pad 8: Net-(R143-Pad1) -> Net-(C36-Pad2)
- U14 pad 4: Net-(R195-Pad1) -> V1_Motor
- U14 pad 6: V1_Motor -> Net-(R167-Pad2)
- U16 pad 4: Net-(R172-Pad1) -> V2_Motor
- U16 pad 6: V2_Motor -> Net-(R169-Pad2)
- U18 pad 4: Net-(R212-Pad1) -> V3_Motor
- U18 pad 6: V3_Motor -> Net-(R208-Pad2)
- U8 pad 14: Net-(R100-Pad1) -> Net-(C6-Pad2)
- U8 pad 8: Net-(R51-Pad1) -> Net-(C5-Pad2)
Routing:
- net GND: track 827.3 -> 672.3 mm, vias 93 -> 154
- net Net-(J31-Pin_1): track 121.5 -> 0.00 mm
- net GND2: track 1745.5 -> 1658.2 mm, vias 69 -> 72
- net Net-(D25-K): track 0.00 -> 74.3 mm
- net T_OptoTriac: track 6.29 -> 52.6 mm
- net +3.3V: track 458.4 -> 502.2 mm, vias 8 -> 11
- net Net-(C31-Pad2): track 0.00 -> 40.1 mm
- net Net-(C6-Pad2): track 0.00 -> 40.0 mm
- net Net-(R122-Pad1): track 37.6 -> 0.00 mm
- net Net-(C35-Pad2): track 0.00 -> 37.5 mm
- net +15V: track 439.5 -> 474.5 mm, vias 6 -> 22
- net Net-(R123-Pad1): track 34.9 -> 0.00 mm
- net VBUS: track 1155.5 -> 1190.3 mm, vias 4 -> 9
- net Net-(R51-Pad1): track 33.9 -> 0.00 mm
- net Net-(R143-Pad1): track 32.6 -> 0.00 mm
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Other:
- outline, holes or cut-outs redrawn
- board text added: "1"
- board text added: "18V External Input"
- board text added: "Analog Outputs"
- board text added: "Bus Input"
- board text added: "DAC1 Inputs"
- board text added: "DAC2 Inputs"
- board text added: "EMULATOR CURRENT GENERATOR"
- board text added: "EMULATOR VOLTAGE GENERATOR"
- board text added: "Firing Output"
- board text added: "GND 3V3 GND 15V"
- board text added: "Opto Triac Outputs"
- board text added: "PWM Inputs"
- board text added: "Phase Voltage Inputs"
- board text added: "Power In"
- board text added: "Power Out"
- board text added: "R Phase Motor - Line"
- board text added: "R Primary Inp"
- board text added: "S Phase Motor - Line"
- board text added: "S Primary Inp"
- board text added: "T Phase Motor - Line"
- board text added: "T Primary Inp"
- board text added: "V Bus Out"
- board text removed: "ABB EMULATOR"
- board text removed: "CURRENT GENERATOR"
- board text removed: "Current Generator 384x 166 mm 70um 2 layers"
- board text removed: "EMULATOR"
- board text removed: "VOLTAGE GENERATOR"
- board text removed: "Voltage Generator 237 x 194 mm 35um 2 layers"
