File: Cur_Emul/Cur_Emul.kicad_sch (KiCad schematic)
At the start: 61 parts, among them J1 Screw_Terminal_01x01, J10 Screw_Terminal_01x01, J11 Screw_Terminal_01x01, J12 Screw_Terminal_01x01, J13 Screw_Terminal_01x01, J14 Screw_Terminal_01x01, J15 Screw_Terminal_01x01, J16 Screw_Terminal_01x01, J2 Screw_Terminal_01x01, J21 Screw_Terminal_01x01, J22 Screw_Terminal_01x01, J3 Screw_Terminal_01x01, J4 Screw_Terminal_01x01, J5 Screw_Terminal_01x01, J6 Screw_Terminal_01x01, J7 Screw_Terminal_01x01, J8 Screw_Terminal_01x01, J9 Screw_Terminal_01x01, M1 IXTH64N10L2, M10 IRF530, M11 IRF530, M12 IRF530, M2 IXTH64N10L2, M3 IXTH64N10L2, M4 IXTH64N10L2, M5 IXTH64N10L2, M6 IXTH64N10L2, M7 IRF530, M8 IRF530, M9 IRF530, T1 Transformer_1P_2S, T2 Transformer_1P_2S, T3 Transformer_1P_2S

Commit message: updates
Parts:
- R158, R44, R48: footprint Resistor_SMD:R_1206_3216Metric_Pad1.30x1.75mm_HandSolder -> Resistor_THT:R_Axial_DIN0204_L3.6mm_D1.6mm_P7.62mm_Horizontal
- R159, R160, R47: footprint Resistor_SMD:R_1206_3216Metric_Pad1.30x1.75mm_HandSolder -> Resistor_SMD:R_Shunt_Vishay_WSR2_WSR3
Connections:
- net GND: no longer R158.2, R159.2, R160.2, R44.2, R47.2, R48.2
- net R_Prim_H: now also T1.6 (SA); no longer T1.10 (SD)
- net R_Prim_L: now also T1.10 (SD); no longer T1.6 (SA)
- net R_Sec_a: now also T1.1 (AA); no longer T1.5 (AB)
- net R_Sec_b: now also T1.5 (AB); no longer T1.1 (AA)
- net S_Prim_H: now also T3.6 (SA); no longer T3.10 (SD)
- net S_Prim_L: now also T3.10 (SD); no longer T3.6 (SA)
- net S_Sec_a: now also T3.1 (AA); no longer T3.5 (AB)
- net S_Sec_b: now also T3.5 (AB); no longer T3.1 (AA)
- net T_Prim_H: now also T2.6 (SA); no longer T2.10 (SD)
- net T_Prim_L: now also T2.10 (SD); no longer T2.6 (SA)
- net T_Sec_a: now also T2.1 (AA); no longer T2.5 (AB)
- net T_Sec_b: now also T2.5 (AB); no longer T2.1 (AA)
- new net GND2: R158.2, R159.2, R160.2, R44.2, R47.2, R48.2
Other:
- moved on the sheet: T1, T2, T3
Changed lines of the file:
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@@
 	)
 	(junction
-		(at 299.72 186.69)
+		(at 198.12 191.77)
 		(diameter 0)
 		(color 0 0 0 0)
@@
 	)
 	(junction
-		(at 106.68 182.88)
-		(diameter 0)
-		(color 0 0 0 0)
-	)
-	(junction
 		(at 140.97 85.09)
 		(diameter 0)
@@
 	)
 	(junction
-		(at 198.12 191.77)
-		(diameter 0)
-		(color 0 0 0 0)
-	)
-	(junction
 		(at 111.76 69.85)
 		(diameter 0)
@@
 	)
 	(junction
+		(at 299.72 186.69)
+		(diameter 0)
+		(color 0 0 0 0)
+	)
+	(junction
 		(at 140.97 74.93)
 		(diameter 0)
@@
 	)
 	(junction
+		(at 106.68 182.88)
+		(diameter 0)
+		(color 0 0 0 0)
+	)
+	(junction
 		(at 196.85 33.02)
 		(diameter 0)
@@
 	(symbol
 		(lib_id "New_Library:Transformer_1P_2S")
-		(at 208.28 181.61 180)
+		(at 208.28 181.61 0)
+		(mirror y)
 		(unit 1)
 		(exclude_from_sim no)
@@
 		(dnp no)
 		(property "Reference" "T3"
-			(at 210.82 171.958 0)
+			(at 210.82 191.262 0)
 			(effects
 				(font
@@
 		)
 		(property "Value" "Transformer_1P_2S"
-			(at 208.28 168.91 0)
+			(at 208.28 194.31 0)
 			(effects
 				(font
@@
 	)
 	(symbol
-		(lib_id "power:GND")
-		(at 39.37 214.63 0)
-		(unit 1)
-		(exclude_from_sim no)
-		(in_bom yes)
-		(on_board yes)
-		(dnp no)
-		(fields_autoplaced yes)
-		(property "Reference" "#PWR027"
-			(at 39.37 220.98 0)
-			(effects
-				(font
-					(size 1.27 1.27)
-				)
-				(hide yes)
-			)
-		)
-		(property "Value" "GND"
-			(at 39.37 219.71 0)
-			(effects
-				(font
-					(size 1.27 1.27)
-				)
-				(hide yes)
-			)
-		)
-		(property "Footprint" ""
-			(at 39.37 214.63 0)
-			(effects
-				(font
-					(size 1.27 1.27)
-				)
-				(hide yes)
-			)
-		)
-		(property "Datasheet" ""
-			(at 39.37 214.63 0)
-			(effects
-				(font
-					(size 1.27 1.27)
-				)
-				(hide yes)
-			)
-		)
-		(property "Description" "Power symbol creates a global label with name \"GND\" , ground"
-			(at 39.37 214.63 0)
-			(effects
-				(font
-					(size 1.27 1.27)
-				)
-				(hide yes)
-			)
-		)
-		(pin "1"
-		)
-		(instances
-			(project "Cur_Emul"
-				(path "/dc5d512a-495b-491d-b4f8-7c4c083c0e6b"
-					(reference "#PWR027")
-					(unit 1)
-				)
-			)
-		)
-	)
-	(symbol
 		(lib_id "Device:R")
 		(at 311.15 78.74 0)
@@
 			)
 		)
-		(property "Footprint" "Resistor_SMD:R_1206_3216Metric_Pad1.30x1.75mm_HandSolder"
+		(property "Footprint" "Resistor_THT:R_Axial_DIN0204_L3.6mm_D1.6mm_P7.62mm_Horizontal"
 			(at 292.862 203.2 90)
 			(effects
@@
 	(symbol
 		(lib_id "New_Library:Transformer_1P_2S")
-		(at 309.88 184.15 180)
+		(at 309.88 184.15 0)
+		(mirror y)
 		(unit 1)
 		(exclude_from_sim no)
@@
 		(dnp no)
 		(property "Reference" "T2"
-			(at 312.166 175.006 0)
+			(at 312.166 193.294 0)
 			(effects
 				(font
@@
 		)
 		(property "Value" "Transformer_1P_2S"
-			(at 309.88 171.45 0)
+			(at 309.88 196.85 0)
 			(effects
 				(font
@@
 			)
 		)
-		(property "Footprint" "Resistor_SMD:R_1206_3216Metric_Pad1.30x1.75mm_HandSolder"
+		(property "Footprint" "Resistor_THT:R_Axial_DIN0204_L3.6mm_D1.6mm_P7.62mm_Horizontal"
 			(at 193.802 203.2 90)
 			(effects
@@
 			)
 		)
-		(property "Footprint" "Resistor_SMD:R_1206_3216Metric_Pad1.30x1.75mm_HandSolder"
+		(property "Footprint" "Resistor_SMD:R_Shunt_Vishay_WSR2_WSR3"
 			(at 197.612 203.2 90)
 			(effects
@@
 			)
 		)
-		(property "Footprint" "Resistor_SMD:R_1206_3216Metric_Pad1.30x1.75mm_HandSolder"
+		(property "Footprint" "Resistor_THT:R_Axial_DIN0204_L3.6mm_D1.6mm_P7.62mm_Horizontal"
 			(at 102.362 200.66 90)
 			(effects
@@
 			)
 		)
-		(property "Footprint" "Resistor_SMD:R_1206_3216Metric_Pad1.30x1.75mm_HandSolder"
+		(property "Footprint" "Resistor_SMD:R_Shunt_Vishay_WSR2_WSR3"
 			(at 296.672 203.2 90)
 			(effects
@@
 	)
 	(symbol
+		(lib_id "power:GND2")
+		(at 39.37 214.63 0)
+		(unit 1)
+		(exclude_from_sim no)
+		(in_bom yes)
+		(on_board yes)
+		(dnp no)
+		(fields_autoplaced yes)
+		(property "Reference" "#PWR021"
+			(at 39.37 220.98 0)
+			(effects
+				(font
+					(size 1.27 1.27)
+				)
+				(hide yes)
+			)
+		)
+		(property "Value" "GND2"
+			(at 39.37 219.71 0)
+			(effects
+				(font
+					(size 1.27 1.27)
+				)
+			)
+		)
+		(property "Footprint" ""
+			(at 39.37 214.63 0)
+			(effects
+				(font
+					(size 1.27 1.27)
+				)
+				(hide yes)
+			)
+		)
+		(property "Datasheet" ""
+			(at 39.37 214.63 0)
+			(effects
+				(font
+					(size 1.27 1.27)
+				)
+				(hide yes)
+			)
+		)
+		(property "Description" "Power symbol creates a global label with name \"GND2\" , ground"
+			(at 39.37 214.63 0)
+			(effects
+				(font
+					(size 1.27 1.27)
+				)
+				(hide yes)
+			)
+		)
+		(pin "1"
+		)
+		(instances
+			(project "Cur_Emul"
+				(path "/dc5d512a-495b-491d-b4f8-7c4c083c0e6b"
+					(reference "#PWR021")
+					(unit 1)
+				)
+			)
+		)
+	)
+	(symbol
 		(lib_id "Transistor_FET:IRF540N")
 		(at 171.45 179.07 0)
@@
 	(symbol
 		(lib_id "New_Library:Transformer_1P_2S")
-		(at 116.84 180.34 180)
+		(at 116.84 180.34 0)
+		(mirror y)
 		(unit 1)
 		(exclude_from_sim no)
@@
 		(dnp no)
 		(property "Reference" "T1"
-			(at 119.126 171.45 0)
+			(at 119.126 189.23 0)
 			(effects
 				(font
@@
 		)
 		(property "Value" "Transformer_1P_2S"
-			(at 116.84 167.64 0)
+			(at 116.84 193.04 0)
 			(effects
 				(font
@@
 			)
 		)
-		(property "Footprint" "Resistor_SMD:R_1206_3216Metric_Pad1.30x1.75mm_HandSolder"
+		(property "Footprint" "Resistor_SMD:R_Shunt_Vishay_WSR2_WSR3"
 			(at 106.172 200.66 90)
 			(effects

Commit message: updates
Parts:
- added JP23, JP24: SolderJumper_2_Bridged, Jumper:SolderJumper-2_P1.3mm_Bridged2Bar_RoundedPad1.0x1.5mm, symbol Jumper:SolderJumper_2_Bridged
Connections:
- net GND: now also JP23.2 (B), JP24.2 (B)
- net GNDPWR: now also JP23.1 (A), JP24.1 (A)
Changed lines of the file:
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@@
 	)
 	(junction
+		(at 59.69 99.06)
+		(diameter 0)
+		(color 0 0 0 0)
+	)
+	(junction
 		(at 106.68 149.86)
 		(diameter 0)
@@
 	)
 	(junction
+		(at 68.58 99.06)
+		(diameter 0)
+		(color 0 0 0 0)
+	)
+	(junction
 		(at 140.97 74.93)
 		(diameter 0)
@@
 	)
 	(junction
+		(at 59.69 91.44)
+		(diameter 0)
+		(color 0 0 0 0)
+	)
+	(junction
 		(at 111.76 74.93)
 		(diameter 0)
@@
 	)
 	(junction
+		(at 68.58 91.44)
+		(diameter 0)
+		(color 0 0 0 0)
+	)
+	(junction
 		(at 281.94 33.02)
 		(diameter 0)
@@
 	(wire
 		(pts
+			(xy 77.47 91.44) (xy 68.58 91.44)
+		)
+		(stroke
+			(width 0)
+			(type default)
+		)
+	)
+	(wire
+		(pts
 			(xy 208.28 93.98) (xy 208.28 59.69)
 		)
@@
 	(wire
 		(pts
+			(xy 68.58 91.44) (xy 59.69 91.44)
+		)
+		(stroke
+			(width 0)
+			(type default)
+		)
+	)
+	(wire
+		(pts
 			(xy 71.12 57.15) (xy 71.12 33.02)
 		)
@@
 	(wire
 		(pts
+			(xy 68.58 99.06) (xy 59.69 99.06)
+		)
+		(stroke
+			(width 0)
+			(type default)
+		)
+	)
+	(wire
+		(pts
 			(xy 223.52 64.77) (xy 223.52 68.58)
 		)
@@
 	(wire
 		(pts
+			(xy 77.47 99.06) (xy 68.58 99.06)
+		)
+		(stroke
+			(width 0)
+			(type default)
+		)
+	)
+	(wire
+		(pts
 			(xy 208.28 106.68) (xy 227.33 106.68)
 		)
@@
 	)
 	(symbol
+		(lib_id "Jumper:SolderJumper_2_Bridged")
+		(at 77.47 95.25 270)
+		(unit 1)
+		(exclude_from_sim no)
+		(in_bom no)
+		(on_board yes)
+		(dnp no)
+		(property "Reference" "JP24"
+			(at 81.788 95.504 90)
+			(effects
+				(font
+					(size 1.27 1.27)
+				)
+			)
+		)
+		(property "Value" "SolderJumper_2_Bridged"
+			(at 81.28 95.25 0)
+			(effects
+				(font
+					(size 1.27 1.27)
+				)
+				(hide yes)
+			)
+		)
+		(property "Footprint" "Jumper:SolderJumper-2_P1.3mm_Bridged2Bar_RoundedPad1.0x1.5mm"
+			(at 77.47 95.25 0)
+			(effects
+				(font
+					(size 1.27 1.27)
+				)
+				(hide yes)
+			)
+		)
+		(property "Datasheet" "~"
+			(at 77.47 95.25 0)
+			(effects
+				(font
+					(size 1.27 1.27)
+				)
+				(hide yes)
+			)
+		)
+		(property "Description" "Solder Jumper, 2-pole, closed/bridged"
+			(at 77.47 95.25 0)
+			(effects
+				(font
+					(size 1.27 1.27)
+				)
+				(hide yes)
+			)
+		)
+		(pin "2"
+		)
+		(pin "1"
+		)
+		(instances
+			(project "Cur_Emul"
+				(path "/dc5d512a-495b-491d-b4f8-7c4c083c0e6b"
+					(reference "JP24")
+					(unit 1)
+				)
+			)
+		)
+	)
+	(symbol
 		(lib_id "power:VDD")
 		(at 39.37 147.32 0)
@@
 					(unit 1)
 				)
+			)
+		)
+	)
+	(symbol
+		(lib_id "Jumper:SolderJumper_2_Bridged")
+		(at 68.58 95.25 270)
+		(unit 1)
+		(exclude_from_sim no)
+		(in_bom no)
+		(on_board yes)
+		(dnp no)
+		(property "Reference" "JP23"
+			(at 72.898 95.504 90)
+			(effects
+				(font
+					(size 1.27 1.27)
+				)
+			)
+		)
+		(property "Value" "SolderJumper_2_Bridged"
+			(at 72.39 95.25 0)
+			(effects
+				(font
+					(size 1.27 1.27)
+				)
+				(hide yes)
+			)
+		)
+		(property "Footprint" "Jumper:SolderJumper-2_P1.3mm_Bridged2Bar_RoundedPad1.0x1.5mm"
+			(at 68.58 95.25 0)
+			(effects
+				(font
+					(size 1.27 1.27)
+				)
+				(hide yes)
+			)
+		)
+		(property "Datasheet" "~"
+			(at 68.58 95.25 0)
+			(effects
+				(font
+					(size 1.27 1.27)
+				)
+				(hide yes)
+			)
+		)
+		(property "Description" "Solder Jumper, 2-pole, closed/bridged"
+			(at 68.58 95.25 0)
+			(effects
+				(font
+					(size 1.27 1.27)
+				)
+				(hide yes)
+			)
+		)
+		(pin "2"
+		)
+		(pin "1"
+		)
+		(instances
+			(project "Cur_Emul"
+				(path "/dc5d512a-495b-491d-b4f8-7c4c083c0e6b"
+					(reference "JP23")
+					(unit 1)
+				)

Commit message: updates4
Parts:
- C9: value 300uF -> 300uF / 50V
- R10, R11, R12, R14, R15, R16, R18, R19, R20, R22, R23, R24, R3, R4, R6, R7, R8: value R -> 10mR
- R158, R44, R48: value R -> 4R7; footprint Resistor_THT:R_Axial_DIN0204_L3.6mm_D1.6mm_P7.62mm_Horizontal -> Resistor_THT:R_Axial_DIN0411_L9.9mm_D3.6mm_P12.70mm_Horizontal
- R159, R160, R47: value R -> 4R7; footprint Resistor_SMD:R_Shunt_Vishay_WSR2_WSR3 -> Resistor_THT:R_Axial_DIN0411_L9.9mm_D3.6mm_P12.70mm_Horizontal
- R2: value 3 X 0.001R -> 10mR
- R68: value R -> 1R
Other:
- note added: "3 X 0.01R"
- note removed: "3 X 0.001R"
