File: Cur_Emul/InputOutput.kicad_sch (KiCad schematic)
At the start: 93 parts, among them J17 Conn_01x04_Pin, J18 Conn_01x02_Pin, J19 Conn_01x04_Pin, J26 Conn_01x04_Pin, J27 Conn_01x04_Pin, J28 Conn_01x04_Pin, J29 Conn_01x02_Pin, J30 Conn_01x02_Pin, J32 Conn_01x04_Pin, J34 Conn_01x06_Pin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

Commit message: updates
Parts:
- removed J19, J27, J32: Conn_01x04_Pin, Connector_JST:JST_EH_B4B-EH-A_1x04_P2.50mm_Vertical, symbol Connector:Conn_01x04_Pin
- removed J36: Conn_01x06_Pin, Connector_JST:JST_PH_B6B-PH-K_1x06_P2.00mm_Vertical, symbol Connector:Conn_01x06_Pin
- added C53: 100nF, symbol Device:C
- added J19, J27, J32: Conn_01x02_Pin, Connector_Phoenix_GMSTB:PhoenixContact_GMSTBVA_2,5_2-G_1x02_P7.50mm_Vertical, symbol Connector:Conn_01x02_Pin
- added J36: Conn_01x08_Pin, Connector_JST:JST_PH_B8B-PH-K_1x08_P2.00mm_Vertical, symbol Connector:Conn_01x08_Pin
- added R219, R227: 10K, Resistor_THT:R_Axial_DIN0207_L6.3mm_D2.5mm_P7.62mm_Horizontal, symbol Device:R
- added R220, R221, R222, R223, R225, R226, R228, R229, R230, R231: 33K, Resistor_THT:R_Axial_DIN0207_L6.3mm_D2.5mm_P7.62mm_Horizontal, symbol Device:R
- added R224: 220R, Resistor_THT:R_Axial_DIN0207_L6.3mm_D2.5mm_P7.62mm_Horizontal, symbol Device:R
- added TP74, TP75, TP76: TestPoint_Alt, TestPoint:TestPoint_Loop_D1.80mm_Drill1.0mm_Beaded, symbol Connector:TestPoint_Alt
- added U21, U22, U23: SFH6206-2T, Package_DIP:SMDIP-4_W9.53mm_Clearance8mm, symbol Isolator:SFH6206-2T
- R171, R172: value 10K -> 220R
- R193: value 470K -> 10K; footprint Resistor_THT:R_Axial_DIN0207_L6.3mm_D2.5mm_P7.62mm_Horizontal -> (none)
- R194, R195, R212: value 470K -> 220R
- R200, R208, R210: value 470K -> 10K
- R202, R204: value 470K -> 33K
Connections:
- net Notr: now also R212.2; no longer R168.2, R170.2, R200.2, R208.2
- net R_Sec_b: now also R171.1; no longer U14.6
- net S_Sec_b: now also R194.1; no longer U16.6
- net T_Sec_b: now also R224.1; no longer U18.6
- net at R177.2: now also J37.1 (Pin_1); no longer R178.1
- net at R189.1: now also U20.2; no longer R188.2
- net at U19.2: now also R184.1; no longer J38.1 (Pin_1)
- net at R204.2: now also J27.1 (Pin_1); no longer R202.1
- net at U16.4: now also R172.1; no longer R169.1
- net at R183.2: now also J38.1 (Pin_1); no longer R184.1
- net at R202.2: now also R204.1; no longer R200.1
- net at R210.1: now also R208.2; no longer R212.2
- net V3_Line: now reaches R208.1
- net V3_Line: now also R224.2; no longer R210.2
- net at U17.2: now also R178.1; no longer J37.1 (Pin_1)
- net at U18.4: now also R212.1; no longer R171.1
- net at J39.1 (Pin_1): now also R188.2; no longer U20.2
- net at U14.4: now also R195.1; no longer R167.1
- net V1_Line: now reaches R171.2
- net V1_Line: now also R167.1; no longer R172.1
- net at R193.2: no longer R194.1
- net V2_Line: now reaches R194.2
- net V2_Line: now also R169.1; no longer R195.1
- net +3.3V renamed +3.3VA
- net +3.3VA: now also R200.2, J36.8 (Pin_8), R219.2, R227.2
- net GND renamed GND2
- net GND2: now also J36.1 (Pin_1), U21.3, U22.3, U23.3; no longer R193.1, R204.1, R212.1
- net R_Phase_Ret renamed R1_Fire
- net R1_Fire: now also J36.2 (Pin_2)
- net S_Phase_Ret renamed S1_Fire
- net S1_Fire: now also J36.4 (Pin_4)
- net T_Phase_Ret renamed T1_Fire
- net T1_Fire: now also J36.6 (Pin_6)
- new net: R225.2, R226.1
- new net: J27.2 (Pin_2), R226.2
- new net: J32.1 (Pin_1), R229.2
- new net: J32.2 (Pin_2), R231.2
- new net: R228.1, U23.1
- new net: R230.1, U23.2
- new net: R220.1, U21.1
- new net: R220.2, R221.1
- new net: J19.1 (Pin_1), R221.2
- new net: J19.2 (Pin_2), R223.2
- new net: R230.2, R231.1
- new net: R202.1, U22.1
- new net: C53.2, R193.1
- new net: R225.1, U22.2
- new net: R228.2, R229.1
- new net: R222.2, R223.1
- new net: R222.1, U21.2
- new net R2_Fire: J36.3 (Pin_3), R219.1, TP74.1, U21.4
- new net S2_Fire: J36.5 (Pin_5), R200.1, TP75.1, U22.4
- new net T2_Fire: J36.7 (Pin_7), R227.1, TP76.1, U23.4
- new net V1_Motor: R168.2, U14.6
- new net V2_Motor: R170.2, U16.6
- new net V3_Motor: R210.2, U18.6
Other:
- note added: "11/17 mA"
- note added: "2V"
- note added: "Fire Detect R1"
- note added: "Fire Detect R2"
- note added: "Fire Detect S1"
- note added: "Fire Detect S2"
- note added: "Fire Detect T1"
- note added: "Fire Detect T2"
- note added: "L1 G K"
- note added: "L2 G K"
- note added: "L3 G K"
- note added: "Phase Voltage Inputs to uc"
- note added: "Snubber !"
- note added: "T1 G K"
- note added: "T2 G K"
- note added: "T3 G K"
- note added: "Thy_L1_Meas"
- note added: "Thy_L2_Meas"
- note added: "Thy_L3_Meas"
- note added: "Thy_T1_Meas"
- note added: "Thy_T2_Meas"
- note added: "Thy_T3_Meas"
- note added: "Thyristor V. Drop Simulation Vdrm 2Volt"
- note added: "To Soft Start Motor Inputs"
- note added: "To Soft Start Phase Voltage Inputs"
- note added: "Transformer Output Sel for Delta/Star Output 220V / 380V"
- moved on the sheet: C50, C51, C52, J17, J18, J26, J28, J29, J30, J34, J37, J38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

Commit message: updates
Parts:
- added J56, J57, J58, J59, J60, J61, J62, J63, J64, J65, J66, J67: Conn_01x01_Pin, Connector_PinHeader_2.54mm:PinHeader_1x01_P2.54mm_Vertical, symbol Connector:Conn_01x01_Pin
- added TP77, TP78: TestPoint_Alt, TestPoint:TestPoint_Loop_D1.80mm_Drill1.0mm_Beaded, symbol Connector:TestPoint_Alt
- J19, J27, J32, J37, J38, J39: footprint Connector_Phoenix_GMSTB:PhoenixContact_GMSTBVA_2,5_2-G_1x02_P7.50mm_Vertical -> Connector_Phoenix_GMSTB:PhoenixContact_GMSTBA_2,5_2-G_1x02_P7.50mm_Horizontal
Connections:
- net +3.3VA: now also J36.1 (Pin_1); no longer J36.8 (Pin_8)
- net GND2: now also J36.8 (Pin_8), TP77.1, TP78.1; no longer J36.1 (Pin_1)
- net R1_Fire: now also J36.7 (Pin_7); no longer J36.2 (Pin_2)
- net R2_Fire: now also J36.6 (Pin_6); no longer J36.3 (Pin_3)
- net R_Prim_H: now also J65.1 (Pin_1)
- net R_Prim_L: now also J64.1 (Pin_1)
- net R_Sec_a: now also J67.1 (Pin_1)
- net R_Sec_b: now also J66.1 (Pin_1)
- net S1_Fire: now also J36.5 (Pin_5); no longer J36.4 (Pin_4)
- net S2_Fire: now also J36.4 (Pin_4); no longer J36.5 (Pin_5)
- net S_Prim_H: now also J61.1 (Pin_1)
- net S_Prim_L: now also J60.1 (Pin_1)
- net S_Sec_a: now also J62.1 (Pin_1)
- net S_Sec_b: now also J63.1 (Pin_1)
- net T1_Fire: now also J36.3 (Pin_3); no longer J36.6 (Pin_6)
- net T2_Fire: now also J36.2 (Pin_2); no longer J36.7 (Pin_7)
- net T_Prim_H: now also J57.1 (Pin_1)
- net T_Prim_L: now also J56.1 (Pin_1)
- net T_Sec_a: now also J58.1 (Pin_1)
- net T_Sec_b: now also J59.1 (Pin_1)
Other:
- note added: "R Grid Volt"
- note added: "S Grid Volt"
- note added: "S Opto Out"
- note added: "T Grid Volt"
- note added: "T Opto Out"
- moved on the sheet: C53, J36, R193

Commit message: with Fabr. Outputs
Parts:
- removed C53: 100nF, symbol Device:C
- removed R171, R194, R224: 220R, Resistor_THT:R_Axial_DIN0207_L6.3mm_D2.5mm_P7.62mm_Horizontal, symbol Device:R
- removed R193: 10K, symbol Device:R
- removed U14, U16, U18: TLP3023, Package_DIP:Toshiba_11-7A9, symbol Isolator:TLP3023
- added J68, J69, J70: 2x7.50mm_Vertical_PhoenixContact_GMSTB, Connector_Phoenix_GMSTB:PhoenixContact_GMSTBVA_2,5_2-G_1x02_P7.50mm_Vertical, symbol Connector:Conn_01x02_Pin
- added U14, U16, U18: MOC3023M, Package_DIP:DIP-6_W7.62mm, symbol Relay_SolidState:MOC3023M
- C50, C51, C52: value 100nF -> 100nF/50V
- J17, J26, J28: value Conn_01x04_Pin -> Conn_01x04_Pin_JST_2.5mm
- J18, J29, J30: value Conn_01x02_Pin -> 2x7.50mm_Vertical_PhoenixContact_GMSTB
- J19, J27, J32, J37, J38, J39: value Conn_01x02_Pin -> 2x7.50mm_Horizontal_PhoenixContact_GMSTBA
- J34: value Conn_01x06_Pin -> Conn_01x06_Pin_JST_2.0mm
- J35: value Conn_01x04_Pin -> Conn_01x04_Pin_JST_2.0mm
- J36: value Conn_01x08_Pin -> Conn_01x08_Pin_JST_2.0mm
- J40, J41, J42, J43, J44, J45, J46, J47, J48, J56, J57, J58, J59, J60, J61, J62, J63, J64, J65, J66, J67: value Conn_01x01_Pin -> PinHeader_1x2.54mm
- R167, R169, R208: value 10K -> 100R
- R168, R170, R210: value 10K -> 100K
- R172, R195, R212: value 220R -> 100K
- R173, R174, R175: footprint Resistor_SMD:R_0805_2012Metric_Pad1.20x1.40mm_HandSolder -> Resistor_THT:R_Axial_DIN0207_L6.3mm_D2.5mm_P7.62mm_Horizontal
- TP61, TP62, TP63, TP64, TP65, TP66, TP67, TP68, TP69, TP70, TP71, TP72, TP74, TP75, TP76, TP77, TP78: value TestPoint_Alt -> Test_Point_THT_KeyStone
- U17, U19, U20, U21, U22, U23: value SFH6206-2T -> SFH620A-2; footprint Package_DIP:SMDIP-4_W9.53mm_Clearance8mm -> Package_DIP:DIP-4_W7.62mm
Connections:
- net V1_Line is gone; now on net R_Sec_b: R167.1
- net V2_Line is gone; now on net S_Sec_b: R169.1
- net V3_Line is gone; now on net T_Sec_b: R208.1
- net GND2: now also J34.6 (Pin_6), U14.2, U16.2, U18.2
- net Notr: now also R168.2, R170.2, R210.2; no longer R172.2, R195.2, R212.2
- net R_Sec_b: now also J70.2 (Pin_2)
- net S_Sec_b: now also J69.2 (Pin_2)
- net T_Sec_b: now also J68.2 (Pin_2)
- net V1_Motor: now also R195.1, J70.1 (Pin_1), U14.4; no longer R168.2
- net V2_Motor: now also R172.1, J69.1 (Pin_1), U16.4; no longer R170.2
- net V3_Motor: now also R212.1, J68.1 (Pin_1), U18.4; no longer R210.2
- net at R170.1: now also R172.2; no longer R169.2
- net at R174.1, TP62.1: now also U16.1
- net at R173.1, TP61.1: now also U14.1
- net at R208.2: now also U18.6; no longer R210.1
- net at R175.1, TP63.1: now also U18.1
- net at R168.1: now also R195.2; no longer R167.2
- new net: R169.2, U16.6
- new net: R210.1, R212.2
- new net: R167.2, U14.6
Other:
- note added: "(Grid - Vthy) Vdrop Around 216 Vac"
- note added: "(Grid-Vmot) Vdrop Around 4Vac"
- note added: "0V"
- note added: "220 Vac"
- note added: "220Vac"
- note added: "4Vdc Vdrop"
- note added: "C"
- note added: "Current Path"
- note added: "Grid"
- note added: "I. and II. Quadrant"
- note added: "III. and IV. Quadrant"
- note added: "Motor"
- note added: "Motor Winding"
- note added: "Motor Winding Voltage Drop Simulation"
- note added: "PSTX Input R"
- note added: "PSTX Input S"
- note added: "PSTX Input T"
- note added: "Snubber"
- note added: "Swing 0- 100 Vac"
- note added: "Thyristors @ Blocking State"
- note added: "Thyristors @ Conducting State"
- moved on the sheet: R167, R168, R169, R170, R173, R208, R210
