File: Cur_Emul/P_Supply.kicad_sch (KiCad schematic)
At the start: 52 parts, among them J31 Conn_01x02_Pin, U13 LM317_SOT-223, U15 LM7812_TO220, U7 LM317_SOT-223

Commit message: updates
Parts:
- removed C37, C38, C39, C40, C45: C_Polarized, Capacitor_SMD:CP_Elec_4x3.9, symbol Device:C_Polarized
- removed C41, C42, C43, C44, C46: C_Polarized, Capacitor_SMD:C_0805_2012Metric_Pad1.18x1.45mm_HandSolder, symbol Device:C
- removed D1: NRVA4004T3G, Diode_SMD:D_SMA, symbol Diode:NRVA4004T3G
- removed D2: LED, LED_SMD:LED_0805_2012Metric_Pad1.15x1.40mm_HandSolder, symbol Device:LED
- removed R161, R164: 1K, Resistor_SMD:R_0805_2012Metric_Pad1.20x1.40mm_HandSolder, symbol Device:R
- added D1: 1N4007, Diode_THT:D_DO-41_SOD81_P10.16mm_Horizontal, symbol Diode:1N4007
- added J49, J50: Conn_01x04_Pin, Connector_Phoenix_GMSTB:PhoenixContact_GMSTBA_2,5_4-G-7,62_1x04_P7.62mm_Horizontal, symbol Connector:Conn_01x04_Pin
- added J51, J52, J53, J54: Conn_01x02_Pin, Connector_Phoenix_GMSTB:PhoenixContact_GMSTBA_2,5_2-G_1x02_P7.50mm_Horizontal, symbol Connector:Conn_01x02_Pin
- added TP73: TestPoint_Alt, TestPoint:TestPoint_Loop_D1.80mm_Drill1.0mm_Beaded, symbol Connector:TestPoint_Alt
- C48: footprint Capacitor_SMD:CP_Elec_6.3x7.7 -> Capacitor_THT:CP_Radial_D24.0mm_P10.00mm_SnapIn
Connections:
- net +15V: now also C3.1, R156.2, R162.2, TP38.1, U7.2 (VO), J49.4 (Pin_4); no longer C47.1, R155.2, R163.2, TP59.1, U13.2 (VO)
- net +3.3V: now also C47.1, R155.2, R163.2, TP59.1, U13.2 (VO), J49.2 (Pin_2); no longer C3.1, R156.2, R162.2, TP38.1, U7.2 (VO)
- net GND: now also J49.1 (Pin_1), J49.3 (Pin_3), J53.2 (Pin_2), J54.2 (Pin_2); no longer C48.2, D17.1 (K), U15.2 (GND), U7.1 (ADJ)
- net VBUS: now also J53.1 (Pin_1), TP73.1; no longer JP21.3 (B)
- net VDD: now also D1.2 (A)
- net at C49.1, J31.1 (Pin_1), JP11.1 (A)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: now also J54.1 (Pin_1); no longer JP21.1 (A)
- net at JP21.2 (C), U15.1 (VI): now also D1.1 (K)
- net at R156.1, R157.2: now also U7.1 (ADJ)
- new net: J52.1 (Pin_1), JP21.3 (B)
- new net: J51.1 (Pin_1), JP21.1 (A)
- new net +12VA: J50.4 (Pin_4)
- new net +3.3VA: J50.2 (Pin_2)
- new net GND2: C48.2, J50.1 (Pin_1), J50.3 (Pin_3), J51.2 (Pin_2), J52.2 (Pin_2), U15.2 (GND)
- new net GNDPWR: D17.1 (K)
Other:
- note added: "BUS INPUT"
- note removed: "Opamp Bypass Voltage Generator 5x 10uF+10nF"
- moved on the sheet: C48, D3, JP21, R162, TP37, TP60, U15

Commit message: updates
Parts:
- added J55: Conn_01x02_Pin, Connector_Phoenix_GMSTB:PhoenixContact_GMSTBA_2,5_2-G_1x02_P7.50mm_Horizontal, symbol Connector:Conn_01x02_Pin
Connections:
- net GND: now also J55.2 (Pin_2)
- net at C49.1, J31.1 (Pin_1), J54.1 (Pin_1)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: now also J55.1 (Pin_1)
Changed lines of the file:
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@@
 	)
 	(junction
+		(at 49.53 130.81)
+		(diameter 0)
+		(color 0 0 0 0)
+	)
+	(junction
 		(at 88.9 107.95)
 		(diameter 0)
@@
 	(wire
 		(pts
+			(xy 63.5 130.81) (xy 49.53 130.81)
+		)
+		(stroke
+			(width 0)
+			(type default)
+		)
+	)
+	(wire
+		(pts
 			(xy 109.22 31.75) (xy 111.76 31.75)
 		)
@@
 	(wire
 		(pts
+			(xy 49.53 130.81) (xy 49.53 113.03)
+		)
+		(stroke
+			(width 0)
+			(type default)
+		)
+	)
+	(wire
+		(pts
 			(xy 64.77 116.84) (xy 78.74 116.84)
 		)
@@
 	(wire
 		(pts
-			(xy 49.53 139.7) (xy 49.53 113.03)
+			(xy 49.53 139.7) (xy 49.53 130.81)
 		)
 		(stroke
@@
 	(wire
 		(pts
+			(xy 63.5 139.7) (xy 63.5 130.81)
+		)
+		(stroke
+			(width 0)
+			(type default)
+		)
+	)
+	(wire
+		(pts
 			(xy 44.45 168.91) (xy 31.75 168.91)
 		)
@@
 	(wire
 		(pts
+			(xy 63.5 144.78) (xy 63.5 142.24)
+		)
+		(stroke
+			(width 0)
+			(type default)
+		)
+	)
+	(wire
+		(pts
 			(xy 55.88 107.95) (xy 57.15 107.95)
 		)
@@
 	(symbol
 		(lib_id "power:GND")
+		(at 63.5 144.78 0)
+		(unit 1)
+		(exclude_from_sim no)
+		(in_bom yes)
+		(on_board yes)
+		(dnp no)
+		(fields_autoplaced yes)
+		(property "Reference" "#PWR0164"
+			(at 63.5 151.13 0)
+			(effects
+				(font
+					(size 1.27 1.27)
+				)
+				(hide yes)
+			)
+		)
+		(property "Value" "GND"
+			(at 63.5 149.86 0)
+			(effects
+				(font
+					(size 1.27 1.27)
+				)
+				(hide yes)
+			)
+		)
+		(property "Footprint" ""
+			(at 63.5 144.78 0)
+			(effects
+				(font
+					(size 1.27 1.27)
+				)
+				(hide yes)
+			)
+		)
+		(property "Datasheet" ""
+			(at 63.5 144.78 0)
+			(effects
+				(font
+					(size 1.27 1.27)
+				)
+				(hide yes)
+			)
+		)
+		(property "Description" "Power symbol creates a global label with name \"GND\" , ground"
+			(at 63.5 144.78 0)
+			(effects
+				(font
+					(size 1.27 1.27)
+				)
+				(hide yes)
+			)
+		)
+		(pin "1"
+		)
+		(instances
+			(project "Cur_Emul"
+				(path "/dc5d512a-495b-491d-b4f8-7c4c083c0e6b/a72b4fff-9e65-4cce-9a53-221bff09e74e"
+					(reference "#PWR0164")
+					(unit 1)
+				)
+			)
+		)
+	)
+	(symbol
+		(lib_id "power:GND")
 		(at 246.38 59.69 0)
 		(unit 1)
@@
 					(unit 1)
 				)
+			)
+		)
+	)
+	(symbol
+		(lib_id "Connector:Conn_01x02_Pin")
+		(at 58.42 139.7 0)
+		(unit 1)
+		(exclude_from_sim no)
+		(in_bom yes)
+		(on_board yes)
+		(dnp no)
+		(property "Reference" "J55"
+			(at 59.182 136.144 0)
+			(effects
+				(font
+					(size 1.27 1.27)
+				)
+			)
+		)
+		(property "Value" "Conn_01x02_Pin"
+			(at 59.055 137.16 0)
+			(effects
+				(font
+					(size 1.27 1.27)
+				)
+				(hide yes)
+			)
+		)
+		(property "Footprint" "Connector_Phoenix_GMSTB:PhoenixContact_GMSTBA_2,5_2-G_1x02_P7.50mm_Horizontal"
+			(at 58.42 139.7 0)
+			(effects
+				(font
+					(size 1.27 1.27)
+				)
+				(hide yes)
+			)
+		)
+		(property "Datasheet" "~"
+			(at 58.42 139.7 0)
+			(effects
+				(font
+					(size 1.27 1.27)
+				)
+				(hide yes)
+			)
+		)
+		(property "Description" "Generic connector, single row, 01x02, script generated"
+			(at 58.42 139.7 0)
+			(effects
+				(font
+					(size 1.27 1.27)
+				)
+				(hide yes)
+			)
+		)
+		(pin "2"
+		)
+		(pin "1"
+		)
+		(instances
+			(project "Cur_Emul"
+				(path "/dc5d512a-495b-491d-b4f8-7c4c083c0e6b/a72b4fff-9e65-4cce-9a53-221bff09e74e"
+					(reference "J55")
+					(unit 1)
+				)

Commit message: updates4
Parts:
- added D18, D2, D23: LED, LED_SMD:LED_0805_2012Metric_Pad1.15x1.40mm_HandSolder, symbol Device:LED
- added R161, R164, R215, R216, R217, R218: 5K, Resistor_SMD:R_0805_2012Metric_Pad1.20x1.40mm_HandSolder, symbol Device:R
- added TP17: TestPoint_Alt, TestPoint:TestPoint_Loop_D1.80mm_Drill1.0mm_Beaded, symbol Connector:TestPoint_Alt
Connections:
- net +12VA: now also R215.2
- net +3.3VA: now also R217.2
- net GND2: now also D18.1 (K), D2.1 (K), D23.1 (K), TP17.1
- net VDD: now also R161.2
- new net: D23.2 (A), R218.1
- new net: R217.1, R218.2
- new net: D18.2 (A), R216.1
- new net: R215.1, R216.2
- new net: R161.1, R164.2
- new net: D2.2 (A), R164.1
Other:
- note added: "Current Generator Board"
- note added: "Voltage Generator Board"
- moved on the sheet: C19, C20, C22, C23, C3, C47, C49, D16, D17, D3, J31, J49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

Commit message: with Fabr. Outputs
Parts:
- removed J49, J50: Conn_01x04_Pin, Connector_Phoenix_GMSTB:PhoenixContact_GMSTBA_2,5_4-G-7,62_1x04_P7.62mm_Horizontal, symbol Connector:Conn_01x04_Pin
- added D24, D25, D26: 1N5407, Diode_THT:D_DO-201AD_P15.24mm_Horizontal, symbol Diode:1N5407
- added J72, J73, J80, J81: 2x7.50mm_Horizontal_PhoenixContact_GMSTBA, Connector_Phoenix_GMSTB:PhoenixContact_GMSTBA_2,5_2-G_1x02_P7.50mm_Horizontal, symbol Connector:Conn_01x02_Pin
- C11, C12, C13, C14, C19, C20: value C_Polarized -> 10uF/50V
- C15, C16, C17, C18, C22, C23: value C_Polarized -> 10nF/50V
- C3, C47: value C_Polarized -> 100uF/50V
- C48: value C_Polarized -> 1000uF/50V
- C49: value 1uF MKT -> 1uF/50V MKT
- J31, J51, J52, J53, J54, J55: value Conn_01x02_Pin -> 2x7.50mm_Horizontal_PhoenixContact_GMSTBA
- R154: value 1K22 -> 1K22 / %1
- R155: value 110R -> 110R / %1
- R156: value 450R -> 450R / %1
- R157: value 750R -> 750R / %1
- TP17, TP37, TP38, TP59, TP60, TP73: value TestPoint_Alt -> Test_Point_THT_KeyStone
Connections:
- net +12VA: now also J81.2 (Pin_2)
- net +15V: now also J73.2 (Pin_2)
- net +3.3V: now also J72.2 (Pin_2)
- net +3.3VA: now also J80.2 (Pin_2)
- net GND: now also J72.1 (Pin_1), J73.1 (Pin_1)
- net GND2: now also J80.1 (Pin_1), J81.1 (Pin_1)
- net VBUS: now also J54.1 (Pin_1)
- net at D1.1 (K), U15.1 (VI): now also D24.1 (K); no longer JP21.2 (C)
- net at C49.1, JP11.1 (A), JP22.1 (A)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: now also D25.1 (K), D26.1 (K); no longer J31.1 (Pin_1), J54.1 (Pin_1), J55.1 (Pin_1)
- net at J52.1 (Pin_1): now also JP21.1 (A); no longer JP21.3 (B)
- net at J51.1 (Pin_1): now also JP21.3 (B); no longer JP21.1 (A)
- new net: D24.2 (A), JP21.2 (C)
- new net: D26.2 (A), J55.1 (Pin_1)
- new net: D25.2 (A), J31.1 (Pin_1)
Other:
- moved on the sheet: J31, J51, J52, J54, J55, JP21, R162
