File: Cur_Emul/Signals.kicad_sch (KiCad schematic)
At the start: 149 parts, among them J20 Conn_01x04_Pin, J23 Conn_01x06_Pin, J24 Conn_01x08_Pin, J25 Conn_01x08_Pin, U1 Opamp_Quad, U2 Opamp_Quad, U3 Opamp_Quad, U4 Opamp_Quad, U5 MCP4922-ESL, U6 MCP4922-ESL

Commit message: updates
Parts:
- removed TP17: TestPoint_Alt, TestPoint:TestPoint_Loop_D1.80mm_Drill1.0mm_Beaded, symbol Connector:TestPoint_Alt
Other:
- note added: "R_Analog_Gain"
- note added: "S_Analog_Gain"
- note added: "S_MOS1 Current Free/Limit"
- note added: "S_MOS2 Current Free/Limit"
- note added: "T_Analog_Gain"
- note added: "T_MOS1 Current Free/Limit"
- note added: "T_MOS2 Current Free/Limit"
Changed lines of the file:
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@@
 		(date "2025-09-04")
 	)
+	(text "S_MOS1 Current\n  Free/Limit"
+		(exclude_from_sim no)
+		(at 211.582 73.66 0)
+		(effects
+			(font
+				(size 1.27 1.27)
+			)
+		)
+	)
 	(text "PWM_2_Analog"
 		(exclude_from_sim no)
@@
 		)
 	)
+	(text "R_Analog_Gain"
+		(exclude_from_sim no)
+		(at 191.77 27.94 0)
+		(effects
+			(font
+				(size 1.27 1.27)
+			)
+		)
+	)
+	(text "T_MOS1 Current\n  Free/Limit"
+		(exclude_from_sim no)
+		(at 220.98 124.46 0)
+		(effects
+			(font
+				(size 1.27 1.27)
+			)
+		)
+	)
+	(text "S_Analog_Gain"
+		(exclude_from_sim no)
+		(at 204.47 58.674 0)
+		(effects
+			(font
+				(size 1.27 1.27)
+			)
+		)
+	)
+	(text "T_MOS2 Current\n  Free/Limit"
+		(exclude_from_sim no)
+		(at 232.41 156.972 0)
+		(effects
+			(font
+				(size 1.27 1.27)
+			)
+		)
+	)
+	(text "T_Analog_Gain"
+		(exclude_from_sim no)
+		(at 204.724 134.874 0)
+		(effects
+			(font
+				(size 1.27 1.27)
+			)
+		)
+	)
+	(text "S_MOS2 Current\n  Free/Limit"
+		(exclude_from_sim no)
+		(at 213.614 96.774 0)
+		(effects
+			(font
+				(size 1.27 1.27)
+			)
+		)
+	)
 	(text "DAC_1 Cont. "
 		(exclude_from_sim no)
@@
 	(wire
 		(pts
-			(xy 35.56 269.24) (xy 35.56 271.78)
-		)
-		(stroke
-			(width 0)
-			(type default)
-		)
-	)
-	(wire
-		(pts
 			(xy 127 53.34) (xy 130.81 53.34)
 		)
@@
 	)
 	(symbol
-		(lib_id "Connector:TestPoint_Alt")
-		(at 35.56 269.24 0)
-		(unit 1)
-		(exclude_from_sim no)
-		(in_bom yes)
-		(on_board yes)
-		(dnp no)
-		(property "Reference" "TP17"
-			(at 34.29 263.144 90)
-			(effects
-				(font
-					(size 1.27 1.27)
-				)
-				(justify left)
-			)
-		)
-		(property "Value" "TestPoint_Alt"
-			(at 38.1 267.2079 0)
-			(effects
-				(font
-					(size 1.27 1.27)
-				)
-				(justify left)
-				(hide yes)
-			)
-		)
-		(property "Footprint" "TestPoint:TestPoint_Loop_D1.80mm_Drill1.0mm_Beaded"
-			(at 40.64 269.24 0)
-			(effects
-				(font
-					(size 1.27 1.27)
-				)
-				(hide yes)
-			)
-		)
-		(property "Datasheet" "~"
-			(at 40.64 269.24 0)
-			(effects
-				(font
-					(size 1.27 1.27)
-				)
-				(hide yes)
-			)
-		)
-		(property "Description" "test point (alternative shape)"
-			(at 35.56 269.24 0)
-			(effects
-				(font
-					(size 1.27 1.27)
-				)
-				(hide yes)
-			)
-		)
-		(pin "1"
-		)
-		(instances
-			(project "Cur_Emul"
-				(path "/dc5d512a-495b-491d-b4f8-7c4c083c0e6b/3008488a-b78b-4e12-986e-52b2be71de9b"
-					(reference "TP17")
-					(unit 1)
-				)
-			)
-		)
-	)
-	(symbol
 		(lib_id "power:GND")
 		(at 208.28 265.43 0)
@@
 					(unit 1)
 				)
-			)
-		)
-	)
-	(symbol
-		(lib_id "power:GND")
-		(at 35.56 271.78 0)
-		(unit 1)
-		(exclude_from_sim no)
-		(in_bom yes)
-		(on_board yes)
-		(dnp no)
-		(fields_autoplaced yes)
-		(property "Reference" "#PWR085"
-			(at 35.56 278.13 0)
-			(effects
-				(font
-					(size 1.27 1.27)
-				)
-				(hide yes)
-			)
-		)
-		(property "Value" "GND"
-			(at 35.56 276.86 0)
-			(effects
-				(font
-					(size 1.27 1.27)
-				)
-				(hide yes)
-			)
-		)
-		(property "Footprint" ""
-			(at 35.56 271.78 0)
-			(effects
-				(font
-					(size 1.27 1.27)
-				)
-				(hide yes)
-			)
-		)
-		(property "Datasheet" ""
-			(at 35.56 271.78 0)
-			(effects
-				(font
-					(size 1.27 1.27)
-				)
-				(hide yes)
-			)
-		)
-		(property "Description" "Power symbol creates a global label with name \"GND\" , ground"
-			(at 35.56 271.78 0)
-			(effects
-				(font
-					(size 1.27 1.27)
-				)
-				(hide yes)
-			)
-		)
-		(pin "1"
-		)
-		(instances
-			(project "Cur_Emul"
-				(path "/dc5d512a-495b-491d-b4f8-7c4c083c0e6b/3008488a-b78b-4e12-986e-52b2be71de9b"
-					(reference "#PWR085")
-					(unit 1)
-				)

Commit message: updates
Parts:
- C1, C2, C4: value 1nF -> 100pF
Changed lines of the file:
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@@
 	(text "S_Analog_Gain"
 		(exclude_from_sim no)
-		(at 204.47 58.674 0)
+		(at 194.818 56.388 0)
 		(effects
 			(font
@@
 			)
 		)
-		(property "Value" "1nF"
-			(at 200.914 89.662 0)
+		(property "Value" "100pF"
+			(at 198.628 89.408 0)
 			(effects
 				(font
@@
 		)
 		(property "Description" "OPA4196"
-			(at 184.15 32.004 0)
+			(at 175.006 30.988 0)
 			(effects
 				(font
@@
 		)
 		(property "Description" "OPA4196"
-			(at 184.658 58.42 0)
+			(at 177.546 58.42 0)
 			(effects
 				(font
@@
 			)
 		)
-		(property "Value" "1nF"
+		(property "Value" "100pF"
 			(at 214.63 152.4 0)
 			(effects
@@
 			)
 		)
-		(property "Value" "1nF"
+		(property "Value" "100pF"
 			(at 204.216 46.228 0)
 			(effects

Commit message: updates4
Parts:
- added C54, C55, C56: 1nF, Capacitor_SMD:C_0805_2012Metric_Pad1.18x1.45mm_HandSolder, symbol Device:C
Connections:
- net at R43.1, RV3.1, RV3.2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: now also C54.2
- net at R73.2, RV3.3, U3.9 (-): now also C54.1
- net at R34.2, RV2.1, RV2.2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: now also C55.2
- net at R59.2, RV1.3, U1.9 (-): now also C56.1
- net at R50.2, RV2.3, U2.9 (-): now also C55.1
- net at R29.1, RV1.1, RV1.2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: now also C56.2
Other:
- note added: "T_Gain"
- moved on the sheet: C1, C4, JP12, JP13, JP15, JP2, JP4, JP7, JP8, JP9, R101, R13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

Commit message: with Fabr. Outputs
Parts:
- removed C1, C2, C4: 100pF, Capacitor_SMD:C_0805_2012Metric_Pad1.18x1.45mm_HandSolder, symbol Device:C
- removed R29, R34, R43: 100R, Resistor_SMD:R_0805_2012Metric_Pad1.20x1.40mm_HandSolder, symbol Device:R
- C25, C7, C8: value 10pF -> 10nF/50V
- C26, C27, C28: value 1uF -> 1uF/50V
- C54, C55, C56: value 1nF -> 10nF/50V
- J20: value Conn_01x04_Pin -> Conn_01x04_Pin_JST_2.0mm
- J23: value Conn_01x06_Pin -> Conn_01x06_Pin_JST_2.0mm
- J24, J25: value Conn_01x08_Pin -> Conn_01x08_Pin_JST_2.0mm
- RV1, RV2, RV3: value 10K -> 10K_SMD_Pot
- TP1, TP10, TP11, TP12, TP13, TP14, TP15, TP16, TP18, TP19, TP2, TP20, TP27, TP28, TP29, TP3, TP30, TP4, TP5, TP6, TP7, TP8, TP9: value TestPoint_Alt -> Test_Point_THT_KeyStone
- TP21, TP22, TP23, TP24, TP25, TP26, TP39, TP40: value TestPoint -> Test_Pad_Not_A_Component
- U1, U2, U3, U4: value Opamp_Quad -> Opamp_Quad_OPA_4196
- U3: value Opamp_Quad -> Opamp_Quad_OPA_4196; footprint Library:SOIC-14_3.9x8.7mm_P1.27mm_ilker -> Package_SO:SOIC-14_3.9x8.7mm_P1.27mm
Connections:
- net at C54.2, RV3.1, RV3.2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: now also R41.1, R42.1
- net at R32.1, R33.1: now also C55.2, RV2.1, RV2.2, TP5.1, U2.8
- net at R27.1, R28.1: now also C56.2, RV1.1, RV1.2, TP4.1, U1.8
Other:
- moved on the sheet: RV1
