File: Cur_Emul/Volt_Gen.kicad_sch (KiCad schematic)
At the start: 118 parts, among them J33 Conn_01x08_Pin, U10 Opamp_Quad, U11 Opamp_Quad, U12 Opamp_Quad, U8 Opamp_Quad, U9 Opamp_Quad

Commit message: updates
Parts:
- added C37, C38, C39, C40, C45: C_Polarized, Capacitor_SMD:CP_Elec_4x3.9, symbol Device:C_Polarized
- added C41, C42, C43, C44, C46: C_Polarized, Capacitor_SMD:C_0805_2012Metric_Pad1.18x1.45mm_HandSolder, symbol Device:C
- added D18, D2, D23: LED, LED_SMD:LED_0805_2012Metric_Pad1.15x1.40mm_HandSolder, symbol Device:LED
- added R161, R164, R215, R216, R217, R218: 5K, Resistor_SMD:R_0805_2012Metric_Pad1.20x1.40mm_HandSolder, symbol Device:R
- added TP17: TestPoint_Alt, TestPoint:TestPoint_Loop_D1.80mm_Drill1.0mm_Beaded, symbol Connector:TestPoint_Alt
Connections:
- net S_Volt_PWM_H: now also J33.3 (Pin_3); no longer J33.4 (Pin_4)
- net S_Volt_PWM_L: now also J33.4 (Pin_4); no longer J33.3 (Pin_3)
- net +15V renamed +12VA
- net +12VA: now also C37.1, C38.1, C39.1, C40.1, C41.1, C42.1, C43.1, C44.1, C45.1, C46.1, R215.2
- net +3.3V renamed +3.3VA
- net +3.3VA: now also R217.2
- net GND renamed GND2
- net GND2: now also C37.2, C38.2, C39.2, C40.2, C41.2, C42.2, C43.2, C44.2, C45.2, C46.2, D18.1 (K), D2.1 (K), D23.1 (K), TP17.1
- new net: D23.2 (A), R218.1
- new net: R217.1, R218.2
- new net: D18.2 (A), R216.1
- new net: R215.1, R216.2
- new net: R161.1, R164.2
- new net: D2.2 (A), R164.1
- new net VDD: R161.2
Other:
- note added: "Opamp Bypass Voltage Generator 5x 10uF+10nF"

Commit message: updates2
Other:
- note added: "R_Analog_Gain"
- note added: "R_High_Analog"
- note added: "R_High_Analog_Gain"
- note added: "R_High_I_Limit"
- note added: "R_High_Mosfet"
- note added: "R_High_PWM"
- note added: "R_Low_Analog"
- note added: "R_Low_Analog_Gain"
- note added: "R_Low_I_Limit"
- note added: "R_Low_Mosfet"
- note added: "R_Low_PWM"
- note added: "S_High_Analog"
- note added: "S_High_Analog_Gain"
- note added: "S_High_I_Limit"
- note added: "S_High_Mosfet"
- note added: "S_High_PWM"
- note added: "S_Low_Analog"
- note added: "S_Low_Analog_Gain"
- note added: "S_Low_I_Limit"
- note added: "S_Low_Mosfet"
- note added: "S_Low_PWM"
- note added: "T_High_Analog"
- note added: "T_High_Analog_Gain"
- note added: "T_High_I_Limit"
- note added: "T_High_Mosfet"
- note added: "T_High_PWM"
- note added: "T_Low_Analog"
- note added: "T_Low_Mosfet"
- note added: "T_Low_PWM"

Commit message: updates4
Parts:
- removed D18, D2, D23: LED, LED_SMD:LED_0805_2012Metric_Pad1.15x1.40mm_HandSolder, symbol Device:LED
- removed R161, R164, R215, R216, R217, R218: 5K, Resistor_SMD:R_0805_2012Metric_Pad1.20x1.40mm_HandSolder, symbol Device:R
- removed TP17: TestPoint_Alt, TestPoint:TestPoint_Loop_D1.80mm_Drill1.0mm_Beaded, symbol Connector:TestPoint_Alt
Other:
- note added: "T_Low_Analog_Gain"
- moved on the sheet: R141

Commit message: with Fabr. Outputs
Parts:
- removed R100, R122, R123, R142, R143, R51: 100R, Resistor_SMD:R_0805_2012Metric_Pad1.20x1.40mm_HandSolder, symbol Device:R
- C21, C24, C29, C30, C33, C34: value 1uF -> 1uF/50V
- C31, C32, C35, C36, C5, C6: value 1nF -> 10nF/50V
- C37, C38, C39, C40, C45: value C_Polarized -> 10uF/50V
- C41, C42, C43, C44, C46: value C_Polarized -> 10nF/50V
- J33: value Conn_01x08_Pin -> Conn_01x08_Pin_JST_2.0mm
- RV4, RV5, RV6, RV7, RV8, RV9: value 10K -> 10K_SMD_Pot
- TP31, TP32, TP33, TP34, TP35, TP36, TP41, TP42, TP43, TP44, TP45, TP46, TP47, TP48, TP49, TP50, TP51, TP52, TP53, TP54, TP55, TP56, TP57, TP58: value TestPoint_Alt -> Test_Point_THT_KeyStone
- U10, U11, U12, U8, U9: value Opamp_Quad -> Opamp_Quad_OPA_4196
Connections:
- net GND2: no longer C31.2, C32.2, C35.2, C36.2, C5.2, C6.2
- net at RV7.1, RV7.2, TP48.1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: now also C32.2, R124.1
- net at R121.2, RV7.3, U10.9 (-): now also C32.1
- net at RV4.1, RV4.2, TP31.1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: now also C5.2, R52.1
- net at C5.1: now also R49.2, RV4.3, U8.9 (-); no longer R52.1
- net at RV6.1, RV6.2, TP47.1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: now also C31.2, R125.1
- net at R120.2, RV6.3, U10.13 (-): now also C31.1
- net at R140.2, RV8.3, U11.13 (-): now also C35.1
- net at RV8.1, RV8.2, TP55.1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: now also C35.2, R145.1
- net at RV9.1, RV9.2, TP56.1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: now also C36.2, R144.1
- net at R141.2, RV9.3, U11.9 (-): now also C36.1
- net at R96.2, RV5.3, U8.13 (-): now also C6.1
- net at RV5.1, RV5.2, TP34.1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: now also C6.2, R53.1
Other:
- note removed: "R_Analog_Gain"
- moved on the sheet: C29, C30, C31, C32, C35, C36, C5, C6, JP16, JP17, R110, R111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
